File: KiCAD/arduino.kicad_sch (KiCad schematic)
At the start: 0 parts

Commit message: KiCad arduino sheet: add Si5351A breakout with CLK0 global label
Place Si5351A_Breakout symbol on arduino sheet and wire CLK0 output
as a global label for inter-sheet connection to the VFO sheet.

Co-Authored-By: Claude Sonnet 4.6 <noreply@anthropic.com>
Parts:
- added U1: Si5351A_Breakout, symbol xmitter:Si5351A_Breakout
- added U2: Metro_ESP32S3, symbol xmitter:Metro_ESP32S3
Connections:
- new net Raw_Clock: U1.CLK0
