File: KiCAD/arduino.kicad_sch (KiCad schematic)
At the start: 15 parts, among them J10 Conn_01x02_Pin, J5 ENC_INT, J6 Conn_01x02_Pin, J7 Conn_01x02_Pin, J8 Conn_01x02_Pin, J9 Conn_01x02_Pin, Q4 2N7000, Q5 2N7000, Q6 2N7000, U17 Adafruit_PCF8575_Breakout, U2 Metro_ESP32S3

Commit message: schematic: I2C topology flip + CD14538B heartbeat + pre-layout audit
- Documentation updates for the STEMMA-QT topology flip (MCP4728 upstream
  of Si5351): design_review_7-5-26 C1 marked resolved, build_checklist
  Phase 1 gets the 6-step first-boot procedure, cw_envelope_keyer I2C
  address section rewritten, front_panel_interface signal-chain diagram
  refreshed.
- CD14538B dual retriggerable monostable added to xmitter.kicad_sym
  (PDIP-16, pinout verified against datasheet fig. 1), plus datasheet
  file.
- Arduino sheet: CD14538B heartbeat topology on Q5 HV contactor -- U18
  + R30 470K + C41 1uF timing (t_w ~470 ms), Q7 series FET stack,
  C42/C43 VDD bypass and bulk.
- Pre-layout audit output as Documentation/punch_list_7-6-26.txt (list
  of blockers before PCB layout, ordered by severity).

Co-Authored-By: Claude Opus 4.7 (1M context) <noreply@anthropic.com>
Parts:
- added C41: 1uF, symbol Device:C
- added C42: 100nF, symbol Device:C
- added C43: 10uF, symbol Device:C_Polarized
- added Q7: 2N7000, Package_TO_SOT_THT:TO-92_Inline, symbol Transistor_FET:2N7000
- added R30: 470K, symbol Device:R_US
- added TP11: Heartbeat, Connector_PinHeader_2.54mm:PinHeader_1x01_P2.54mm_Vertical, symbol xmitter:xTP
- added U18: CD14538B, Package_DIP:DIP-16_W7.62mm, symbol xmitter:CD14538B
- J10: value Conn_01x02_Pin -> Paddle
- J6: value Conn_01x02_Pin -> TX/RX
- J7: value Conn_01x02_Pin -> HV
- J8: value Conn_01x02_Pin -> HV_INRUSH_BYPASS
- J9: value Conn_01x02_Pin -> TR_SENSE
Connections:
- net +5V: now also C42.1, C43.1, R30.2, U18.11 (~{RST}_B), U18.12 (+TR_B), U18.16 (VDD), U18.5 (~{RST}_A)
- net GND: now also C42.2, C43.2, Q7.1 (S), U18.13 (-TR_B), U18.3 (-TR_A), U18.8 (VSS); no longer Q5.1 (S)
- net at U17.P12: now also U18.4 (+TR_A)
- net RESET_N: now reaches U2.RESET
- new net: C41.2, R30.1, U18.2 (RC_A)
- new net: Q5.1 (S), Q7.3 (D)
- new net: Q7.2 (G), TP11.1, U18.6 (Q_A)
- new net: C41.1, U18.1 (C_A)
Other:
- note added: "J9 goes to the second set of contacts on the transmit/receive relay. This is the source of TR_SENSE which confirms that the relay is in the correct state. (It switches between GND and +3.3V)"
- note removed: "J8 goes to the second set of contacts on the transmit/receive relay. This is the source of TR_SENSE which confirms that the relay is in the correct state. (It switches between GND and +3.3V)"
- moved on the sheet: J7, J8, Q5, Q6

Commit message: kicad: convert hierarchical labels to globals (Path A) + unify _OUT/_IN pairs
- 58 hierarchical_label -> global_label conversions across the six active
  sheets. Standard KiCad 10 global_label form with fields_autoplaced +
  Intersheetrefs property.
- Stripped 36 vestigial sheet pins, 28 stitching wires, 2 junctions, 4
  labels from the root sheet. Sheet blocks remain; each is now a pure
  container with globals doing the cross-sheet connectivity by name.
- Renamed three OUT/IN pairs to unified names so same-name globals
  auto-connect:
    GRID_CTL_A_OUT + GRID_CTL_A_IN -> GRID_CTL_A
    GRID_CTL_B_OUT + GRID_CTL_B_IN -> GRID_CTL_B
    RAW_RF_OUT     + RAW_RF_IN     -> RAW_RF
- tools/convert_hier_to_global.py and tools/strip_root_stitching.py:
  reusable if we ever need to redo this.
- Documentation/punch_list_7-6-26.txt: mark B1a-e, L1, L2 resolved; add
  M6 (cosmetic) about GRID_CTL_A's label-at-pin-origin idiom; correct
  the earlier GRID_CTL_A false positive with the verified chain
  MCP4728 U8 VC -> R_PADA -> OPA454 U5 IN+ + Q3 drain.

Co-Authored-By: Claude Opus 4.7 (1M context) <noreply@anthropic.com>
Changed lines of the file:
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@@
 		)
 	)
-	(hierarchical_label "CS_DAC"
+	(global_label "CS_DAC"
 		(shape output)
 		(at 119.38 64.77 0)
-		(effects
-			(font
-				(size 1.27 1.27)
-			)
-			(justify left)
-		)
-	)
-	(hierarchical_label "SDA"
+		(fields_autoplaced yes)
+		(effects
+			(font
+				(size 1.27 1.27)
+			)
+			(justify left)
+		)
+		(property "Intersheetrefs" "${INTERSHEET_REFS}"
+			(at 119.38 64.77 0)
+			(effects
+				(font
+					(size 1.27 1.27)
+				)
+				(hide yes)
+			)
+		)
+	)
+	(global_label "SDA"
 		(shape bidirectional)
 		(at 175.26 66.04 180)
-		(effects
-			(font
-				(size 1.27 1.27)
-			)
-			(justify right)
-		)
-	)
-	(hierarchical_label "LDAC_4728"
+		(fields_autoplaced yes)
+		(effects
+			(font
+				(size 1.27 1.27)
+			)
+			(justify right)
+		)
+		(property "Intersheetrefs" "${INTERSHEET_REFS}"
+			(at 175.26 66.04 0)
+			(effects
+				(font
+					(size 1.27 1.27)
+				)
+				(hide yes)
+			)
+		)
+	)
+	(global_label "LDAC_4728"
 		(shape output)
 		(at 88.9 83.82 180)
-		(effects
-			(font
-				(size 1.27 1.27)
-			)
-			(justify right)
-		)
-	)
-	(hierarchical_label "I_CATHODE_B"
+		(fields_autoplaced yes)
+		(effects
+			(font
+				(size 1.27 1.27)
+			)
+			(justify right)
+		)
+		(property "Intersheetrefs" "${INTERSHEET_REFS}"
+			(at 88.9 83.82 0)
+			(effects
+				(font
+					(size 1.27 1.27)
+				)
+				(hide yes)
+			)
+		)
+	)
+	(global_label "I_CATHODE_B"
 		(shape input)
 		(at 88.9 88.9 180)
-		(effects
-			(font
-				(size 1.27 1.27)
-			)
-			(justify right)
-		)
-	)
-	(hierarchical_label "MBL600_B"
+		(fields_autoplaced yes)
+		(effects
+			(font
+				(size 1.27 1.27)
+			)
+			(justify right)
+		)
+		(property "Intersheetrefs" "${INTERSHEET_REFS}"
+			(at 88.9 88.9 0)
+			(effects
+				(font
+					(size 1.27 1.27)
+				)
+				(hide yes)
+			)
+		)
+	)
+	(global_label "MBL600_B"
 		(shape input)
 		(at 88.9 78.74 180)
-		(effects
-			(font
-				(size 1.27 1.27)
-			)
-			(justify right)
-		)
-	)
-	(hierarchical_label "MBL600_A"
+		(fields_autoplaced yes)
+		(effects
+			(font
+				(size 1.27 1.27)
+			)
+			(justify right)
+		)
+		(property "Intersheetrefs" "${INTERSHEET_REFS}"
+			(at 88.9 78.74 0)
+			(effects
+				(font
+					(size 1.27 1.27)
+				)
+				(hide yes)
+			)
+		)
+	)
+	(global_label "MBL600_A"
 		(shape input)
 		(at 88.9 76.2 180)
-		(effects
-			(font
-				(size 1.27 1.27)
-			)
-			(justify right)
-		)
-	)
-	(hierarchical_label "SCL"
+		(fields_autoplaced yes)
+		(effects
+			(font
+				(size 1.27 1.27)
+			)
+			(justify right)
+		)
+		(property "Intersheetrefs" "${INTERSHEET_REFS}"
+			(at 88.9 76.2 0)
+			(effects
+				(font
+					(size 1.27 1.27)
+				)
+				(hide yes)
+			)
+		)
+	)
+	(global_label "SCL"
 		(shape bidirectional)
 		(at 175.26 63.5 180)
-		(effects
-			(font
-				(size 1.27 1.27)
-			)
-			(justify right)
-		)
-	)
-	(hierarchical_label "GRID_BLOCK_CRASH"
+		(fields_autoplaced yes)
+		(effects
+			(font
+				(size 1.27 1.27)
+			)
+			(justify right)
+		)
+		(property "Intersheetrefs" "${INTERSHEET_REFS}"
+			(at 175.26 63.5 0)
+			(effects
+				(font
+					(size 1.27 1.27)
+				)
+				(hide yes)
+			)
+		)
+	)
+	(global_label "GRID_BLOCK_CRASH"
 		(shape input)
 		(at 119.38 72.39 0)
-		(effects
-			(font
-				(size 1.27 1.27)
-			)
-			(justify left)
-		)
-	)
-	(hierarchical_label "SCK"
+		(fields_autoplaced yes)
+		(effects
+			(font
+				(size 1.27 1.27)
+			)
+			(justify left)
+		)
+		(property "Intersheetrefs" "${INTERSHEET_REFS}"
+			(at 119.38 72.39 0)
+			(effects
+				(font
+					(size 1.27 1.27)
+				)
+				(hide yes)
+			)
+		)
+	)
+	(global_label "SCK"
 		(shape output)
 		(at 119.38 69.85 0)
-		(effects
-			(font
-				(size 1.27 1.27)
-			)
-			(justify left)
-		)
-	)
-	(hierarchical_label "I_CATHODE_A"
+		(fields_autoplaced yes)
+		(effects
+			(font
+				(size 1.27 1.27)
+			)
+			(justify left)
+		)
+		(property "Intersheetrefs" "${INTERSHEET_REFS}"
+			(at 119.38 69.85 0)
+			(effects
+				(font
+					(size 1.27 1.27)
+				)
+				(hide yes)
+			)
+		)
+	)
+	(global_label "I_CATHODE_A"
 		(shape input)
 		(at 88.9 86.36 180)
-		(effects
-			(font
-				(size 1.27 1.27)
-			)
-			(justify right)
-		)
-	)
-	(hierarchical_label "RESET_N"
+		(fields_autoplaced yes)
+		(effects
+			(font
+				(size 1.27 1.27)
+			)
+			(justify right)
+		)
+		(property "Intersheetrefs" "${INTERSHEET_REFS}"
+			(at 88.9 86.36 0)
+			(effects
+				(font
+					(size 1.27 1.27)
+				)
+				(hide yes)
+			)
+		)
+	)
+	(global_label "RESET_N"
 		(shape input)
 		(at 88.9 68.58 180)
-		(effects
-			(font
-				(size 1.27 1.27)
-			)
-			(justify right)
-		)
-	)
-	(hierarchical_label "MOSI"
+		(fields_autoplaced yes)
+		(effects
+			(font
+				(size 1.27 1.27)
+			)
+			(justify right)
+		)
+		(property "Intersheetrefs" "${INTERSHEET_REFS}"
+			(at 88.9 68.58 0)
+			(effects
+				(font
+					(size 1.27 1.27)
+				)
+				(hide yes)
+			)
+		)
+	)
+	(global_label "MOSI"
 		(shape output)
 		(at 119.38 67.31 0)
-		(effects
-			(font
-				(size 1.27 1.27)
-			)
-			(justify left)
-		)
-	)
+		(fields_autoplaced yes)
+		(effects
+			(font
+				(size 1.27 1.27)
+			)
+			(justify left)
+		)
+		(property "Intersheetrefs" "${INTERSHEET_REFS}"
+			(at 119.38 67.31 0)
+			(effects
+				(font
+					(size 1.27 1.27)
+				)
+				(hide yes)
+			)
+		)
+	)

Commit message: kicad: fill 9 remaining footprints across active sheets
- arduino: R30 470K (R_Axial_DIN0207 horizontal), C41 1uF (rect L7.2mm),
  C42 100nF (disc D5mm P5mm), C43 10uF (radial polarized D5mm P2mm)
- bias: J11 (GRID_BIAS), J12 (CATHODE_SENSE), J14 -- all PinHeader_1x02
  vertical THT
- buffer_keyer: J13 -- PinHeader_1x05 vertical THT
- interface: J15 -- PinHeader_1x03 vertical THT

C41/C42/C43 filled by re-running tools/assign_cap_footprints.py which
already had the intended mappings. R30 and the connectors done by hand
via a one-off script.

Only U2 (Metro) remains footprint-less, intentionally off-PCB.

Punch list updates for today's ERC pass + user's schematic edits:
- B3 (footprints) resolved.
- B4d/B4e (TP2/TP7 to MOD_RF+/-) resolved -- user verified junction dots
  + wires in KiCad. TP3 = SCL is intentional (I2C debug probe access).
- M5 (TX_LED) previously resolved -- LED wired in parallel with T/R
  relay coil, no Metro GPIO needed.
- B2 (paddle) rewritten for the actual design: J10 = 2-conductor 1/4"
  phone plug, tip -> Metro D5, sleeve -> GND.

vfo.kicad_sch diff is KiCad's own canonicalization of Intersheetrefs
property (show_name/do_not_autoplace fields shuffled) from opening +
saving; contents equivalent.

Co-Authored-By: Claude Opus 4.7 (1M context) <noreply@anthropic.com>
Parts:
- C41: footprint (none) -> Capacitor_THT:C_Rect_L7.2mm_W4.5mm_P5.00mm
- C42: footprint (none) -> Capacitor_THT:C_Disc_D5.0mm_W2.5mm_P5.00mm
- C43: footprint (none) -> Capacitor_THT:CP_Radial_D5.0mm_P2.00mm
- J5: value ENC_INT -> ENC_INT if needed
- R30: footprint (none) -> Resistor_THT:R_Axial_DIN0207_L6.3mm_D2.5mm_P10.16mm_Horizontal
Changed lines of the file:
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@@
 		(property "Intersheetrefs" "${INTERSHEET_REFS}"
 			(at 119.38 64.77 0)
+			(hide yes)
+			(show_name no)
+			(do_not_autoplace no)
 			(effects
 				(font
 					(size 1.27 1.27)
 				)
-				(hide yes)
 			)
 		)
@@
 		(property "Intersheetrefs" "${INTERSHEET_REFS}"
 			(at 175.26 66.04 0)
+			(hide yes)
+			(show_name no)
+			(do_not_autoplace no)
 			(effects
 				(font
 					(size 1.27 1.27)
 				)
-				(hide yes)
 			)
 		)
@@
 		(property "Intersheetrefs" "${INTERSHEET_REFS}"
 			(at 88.9 83.82 0)
+			(hide yes)
+			(show_name no)
+			(do_not_autoplace no)
 			(effects
 				(font
 					(size 1.27 1.27)
 				)
-				(hide yes)
 			)
 		)
@@
 		(property "Intersheetrefs" "${INTERSHEET_REFS}"
 			(at 88.9 88.9 0)
+			(hide yes)
+			(show_name no)
+			(do_not_autoplace no)
 			(effects
 				(font
 					(size 1.27 1.27)
 				)
-				(hide yes)
 			)
 		)
@@
 		(property "Intersheetrefs" "${INTERSHEET_REFS}"
 			(at 88.9 78.74 0)
+			(hide yes)
+			(show_name no)
+			(do_not_autoplace no)
 			(effects
 				(font
 					(size 1.27 1.27)
 				)
-				(hide yes)
 			)
 		)
@@
 		(property "Intersheetrefs" "${INTERSHEET_REFS}"
 			(at 88.9 76.2 0)
+			(hide yes)
+			(show_name no)
+			(do_not_autoplace no)
 			(effects
 				(font
 					(size 1.27 1.27)
 				)
-				(hide yes)
 			)
 		)
@@
 		(property "Intersheetrefs" "${INTERSHEET_REFS}"
 			(at 175.26 63.5 0)
+			(hide yes)
+			(show_name no)
+			(do_not_autoplace no)
 			(effects
 				(font
 					(size 1.27 1.27)
 				)
-				(hide yes)
 			)
 		)
@@
 		(property "Intersheetrefs" "${INTERSHEET_REFS}"
 			(at 119.38 72.39 0)
+			(hide yes)
+			(show_name no)
+			(do_not_autoplace no)
 			(effects
 				(font
 					(size 1.27 1.27)
 				)
-				(hide yes)
 			)
 		)
@@
 		(property "Intersheetrefs" "${INTERSHEET_REFS}"
 			(at 119.38 69.85 0)
+			(hide yes)
+			(show_name no)
+			(do_not_autoplace no)
 			(effects
 				(font
 					(size 1.27 1.27)
 				)
-				(hide yes)
 			)
 		)
@@
 		(property "Intersheetrefs" "${INTERSHEET_REFS}"
 			(at 88.9 86.36 0)
+			(hide yes)
+			(show_name no)
+			(do_not_autoplace no)
 			(effects
 				(font
 					(size 1.27 1.27)
 				)
-				(hide yes)
 			)
 		)
@@
 		(property "Intersheetrefs" "${INTERSHEET_REFS}"
 			(at 88.9 68.58 0)
+			(hide yes)
+			(show_name no)
+			(do_not_autoplace no)
 			(effects
 				(font
 					(size 1.27 1.27)
 				)
-				(hide yes)
 			)
 		)
@@
 		(property "Intersheetrefs" "${INTERSHEET_REFS}"
 			(at 119.38 67.31 0)
+			(hide yes)
+			(show_name no)
+			(do_not_autoplace no)
 			(effects
 				(font
 					(size 1.27 1.27)
 				)
-				(hide yes)
 			)
 		)
@@
 			)
 		)
-		(property "Footprint" ""
+		(property "Footprint" "Resistor_THT:R_Axial_DIN0207_L6.3mm_D2.5mm_P10.16mm_Horizontal"
 			(at 179.324 148.844 90)
 			(hide yes)
@@
 			)
 		)
-		(property "Footprint" ""
+		(property "Footprint" "Capacitor_THT:C_Rect_L7.2mm_W4.5mm_P5.00mm"
 			(at 175.26 146.3548 0)
 			(hide yes)
@@
 			)
 		)
-		(property "Footprint" ""
+		(property "Footprint" "Capacitor_THT:C_Disc_D5.0mm_W2.5mm_P5.00mm"
 			(at 165.1 127.3048 0)
 			(hide yes)
@@
 			)
 		)
-		(property "Value" "ENC_INT"
+		(property "Value" "ENC_INT if needed"
 			(at 56.1974 77.47 0)
 			(show_name no)
@@
 			)
 		)
-		(property "Footprint" ""
+		(property "Footprint" "Capacitor_THT:CP_Radial_D5.0mm_P2.00mm"
 			(at 149.86 129.2352 0)
 			(hide yes)

Commit message: kicad: PWR_FLAGs added, most +3.3V converted to 3V3, VFO renames + J2 NC
User work today:
- Placed PWR_FLAGs to silence "power_pin_not_driven" ERC errors for VEE,
  +12V, -90V rails (see B5a-B5f in the punch list)
- Converted 6 of 7 +3.3V power symbols to 3V3 global labels project-wide
  (one +3.3V remains on bias sheet, resolves next pass)
- VFO sheet: C_coup -> C_IN1, R6 -> RD1 (both were unannotated / duplicate
  ref designators; ERC B4a and B4b now resolved)
- buffer_keyer: J2 pin 2 gets a no_connect flag (B4c resolved); TP2 and
  TP7 electrically wired to MOD_RF_OUT+/- via junctions (B4d/e resolved)

Punch list updates:
- B3 (footprints) marked done
- B4a/b/c marked done
- M5 (TX LED) confirmed resolved (external LED across T/R relay coil)
- B2 (paddle) rewritten for the actual 2-conductor 1/4" plug scheme

Current ERC status: 61 errors, 0 warnings (from 74 + 2 originally).
Remaining real bugs: unannotated C_IN + duplicate C_IN1 on buffer_keyer,
misplaced #FLG04 on Metro's 3V3 pin, one leftover +3.3V on bias. Rest
are the known-non-issue plateau.

Co-Authored-By: Claude Opus 4.7 (1M context) <noreply@anthropic.com>
Connections:
- net +3.3V is gone; now on net 3V3: J9.1 (Pin_1), R102.1
- net 3V3: now reaches U2.3V3_L (3V3)
- no-connect marks 2 -> 13
Changed lines of the file:
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@@
 	)
 	(no_connect
+		(at 88.9 66.04)
+	)
+	(no_connect
+		(at 119.38 74.93)
+	)
+	(no_connect
+		(at 167.64 162.56)
+	)
+	(no_connect
+		(at 167.64 154.94)
+	)
+	(no_connect
 		(at 88.9 73.66)
 	)
 	(no_connect
+		(at 119.38 85.09)
+	)
+	(no_connect
 		(at 88.9 71.12)
 	)
+	(no_connect
+		(at 119.38 80.01)
+	)
+	(no_connect
+		(at 119.38 77.47)
+	)
+	(no_connect
+		(at 167.64 165.1)
+	)
+	(no_connect
+		(at 119.38 82.55)
+	)
+	(no_connect
+		(at 167.64 142.24)
+	)
+	(no_connect
+		(at 167.64 157.48)
+	)
 	(wire
 		(pts
@@
 	(wire
 		(pts
-			(xy 135.89 90.17) (xy 137.16 90.17)
+			(xy 224.79 109.22) (xy 224.79 113.03)
 		)
 		(stroke
@@
 	(wire
 		(pts
-			(xy 224.79 109.22) (xy 224.79 113.03)
+			(xy 175.26 147.32) (xy 175.26 149.86)
 		)
 		(stroke
@@
 	(wire
 		(pts
-			(xy 175.26 147.32) (xy 175.26 149.86)
+			(xy 69.85 63.5) (xy 88.9 63.5)
 		)
 		(stroke
@@
 	(wire
 		(pts
+			(xy 73.66 71.12) (xy 73.66 73.66)
+		)
+		(stroke
+			(width 0)
+			(type default)
+		)
+	)
+	(wire
+		(pts
+			(xy 133.35 90.17) (xy 137.16 90.17)
+		)
+		(stroke
+			(width 0)
+			(type default)
+		)
+	)
+	(wire
+		(pts
 			(xy 123.19 87.63) (xy 119.38 87.63)
 		)
@@
 		)
 	)
+	(global_label "3V3"
+		(shape input)
+		(at 73.66 71.12 90)
+		(fields_autoplaced yes)
+		(effects
+			(font
+				(size 1.27 1.27)
+			)
+			(justify left)
+		)
+		(property "Intersheetrefs" "${INTERSHEET_REFS}"
+			(at 73.66 64.6272 90)
+			(hide yes)
+			(show_name no)
+			(do_not_autoplace no)
+			(effects
+				(font
+					(size 1.27 1.27)
+				)
+				(justify left)
+			)
+		)
+	)
 	(global_label "SDA"
 		(shape bidirectional)
@@
 		)
 	)
+	(global_label "3V3"
+		(shape input)
+		(at 133.35 90.17 180)
+		(fields_autoplaced yes)
+		(effects
+			(font
+				(size 1.27 1.27)
+			)
+			(justify right)
+		)
+		(property "Intersheetrefs" "${INTERSHEET_REFS}"
+			(at 126.8572 90.17 0)
+			(hide yes)
+			(show_name no)
+			(do_not_autoplace no)
+			(effects
+				(font
+					(size 1.27 1.27)
+				)
+				(justify right)
+			)
+		)
+	)
 	(global_label "MBL600_A"
 		(shape input)
@@
 		)
 	)
+	(global_label "3V3"
+		(shape output)
+		(at 69.85 63.5 180)
+		(fields_autoplaced yes)
+		(effects
+			(font
+				(size 1.27 1.27)
+			)
+			(justify right)
+		)
+		(property "Intersheetrefs" "${INTERSHEET_REFS}"
+			(at 63.3572 63.5 0)
+			(hide yes)
+			(show_name no)
+			(do_not_autoplace no)
+			(effects
+				(font
+					(size 1.27 1.27)
+				)
+				(justify right)
+			)
+		)
+	)
 	(global_label "RESET_N"
 		(shape input)
@@
 	)
 	(symbol
-		(lib_id "power:+3.3V")
-		(at 135.89 90.17 90)
-		(unit 1)
-		(body_style 1)
-		(exclude_from_sim no)
-		(in_bom yes)
-		(on_board yes)
-		(in_pos_files yes)
-		(dnp no)
-		(fields_autoplaced yes)
-		(property "Reference" "#PWR0110"
-			(at 139.7 90.17 0)
-			(hide yes)
-			(show_name no)
-			(do_not_autoplace no)
-			(effects
-				(font
-					(size 1.27 1.27)
-				)
-			)
-		)
-		(property "Value" "+3.3V"
-			(at 132.08 90.1699 90)
-			(show_name no)
-			(do_not_autoplace no)
-			(effects
-				(font
-					(size 1.27 1.27)
-				)
-				(justify left)
-			)
-		)
-		(property "Footprint" ""
-			(at 135.89 90.17 0)
-			(hide yes)
-			(show_name no)
-			(do_not_autoplace no)
-			(effects
-				(font
-					(size 1.27 1.27)
-				)
-			)
-		)
-		(property "Datasheet" ""
-			(at 135.89 90.17 0)
-			(hide yes)
-			(show_name no)
-			(do_not_autoplace no)
-			(effects
-				(font
-					(size 1.27 1.27)
-				)
-			)
-		)
-		(property "Description" "Power symbol creates a global label with name \"+3.3V\""
-			(at 135.89 90.17 0)
-			(hide yes)
-			(show_name no)
-			(do_not_autoplace no)
-			(effects
-				(font
-					(size 1.27 1.27)
-				)
-			)
-		)
-		(pin "1"
-		)
-		(instances
-			(project "KiCAD"
-				(path "/d3de40b8-856b-4fbd-829c-f45ffcd55742/2d83d0b5-86d4-4ced-ab68-6465e3dc2d72"
-					(reference "#PWR0110")
-					(unit 1)
-				)
-			)
-		)
-	)
-	(symbol
 		(lib_id "xmitter:CD14538B")
 		(at 157.48 152.4 0)
@@
 					(unit 1)
 				)
-			)
-		)
-	)
-	(symbol
-		(lib_id "power:+3.3V")
-		(at 73.66 73.66 0)
-		(unit 1)
-		(body_style 1)
-		(exclude_from_sim no)
-		(in_bom yes)
-		(on_board yes)
-		(in_pos_files yes)
-		(dnp no)
-		(fields_autoplaced yes)
-		(property "Reference" "#PWR100"
-			(at 73.66 77.47 0)
-			(hide yes)
-			(show_name no)
-			(do_not_autoplace no)
-			(effects
-				(font
-					(size 1.27 1.27)
-				)
-			)
-		)
-		(property "Value" "+3.3V"
-			(at 73.66 69.85 0)
-			(show_name no)
-			(do_not_autoplace no)
-			(effects
-				(font
-					(size 1.27 1.27)
-				)
-			)
-		)
-		(property "Footprint" ""
-			(at 73.66 73.66 0)
-			(hide yes)
-			(show_name no)
-			(do_not_autoplace no)
-			(effects
-				(font
-					(size 1.27 1.27)
-				)
-			)
-		)
-		(property "Datasheet" ""
-			(at 73.66 73.66 0)
-			(hide yes)
-			(show_name no)
-			(do_not_autoplace no)
-			(effects
-				(font
-					(size 1.27 1.27)
-				)
-			)
-		)
-		(property "Description" "Power symbol creates a global label with name \"+3.3V\""
-			(at 73.66 73.66 0)
-			(hide yes)
-			(show_name no)
-			(do_not_autoplace no)
-			(effects
-				(font
-					(size 1.27 1.27)
-				)
-			)
-		)
-		(pin "1"
-		)
-		(instances
-			(project "KiCAD"
-				(path "/d3de40b8-856b-4fbd-829c-f45ffcd55742/2d83d0b5-86d4-4ced-ab68-6465e3dc2d72"
-					(reference "#PWR100")
-					(unit 1)
-				)
