File: KiCAD/vfo.kicad_sch (KiCad schematic)
At the start: 0 parts

Commit message: Work in Progress
Parts:
- added C1, C4: 200pF, symbol Device:C
- added C3: 360pF, symbol Device:C
- added L1, L2: 624nH, symbol Device:L_Ferrite
- added Q1: J310, Package_TO_SOT_THT:TO-92_Inline, symbol xmitter:J310
- added R1, R5: 50R, symbol Device:R_US
- added R2, R4: 150R, symbol Device:R_US
- added R3: 39R, symbol Device:R_US
- added R6: 270R, symbol Device:R_US
- added U3: MC1496, Package_DIP:DIP-14_W7.62mm, symbol xmitter:MC1496
Connections:
- new net: Q1.1 (S), R6.1
- new net: C4.1, L2.2, Q1.2 (G), R5.1
- new net: C3.1, L1.2, L2.1
- new net: R1.2, R2.1, R3.2
- new net: C1.1, L1.1, R3.1, R4.1
- new net +12V: Q1.3 (D)
- new net GND: C1.2, C3.2, C4.2, R2.2, R4.2, R5.2, R6.2
- new net Raw Clock: R1.1
