File: KiCAD/vfo.kicad_sch (KiCad schematic)
At the start: 17 parts, among them Q1 J310, U1 Si5351A_Breakout

Commit message: kicad(bias): build complete grid-bias sheet (Design A: dual OPA454)
New sheet untitled.kicad_sch (sheet name "Bias", file to be renamed
bias.kicad_sch) implementing the OPA454 high-voltage design per the
Grid_Bias_Schematic.pdf design doc:

- LM7805 (U9) generates the +5 V supply rail from +12 V (~30 mA load,
  no heatsink needed at ~270 mW dissipation)
- LM4040DIZ-5.0 (U11) generates a SEPARATE +5 V_REF precision reference
  biased from +12 V via R_Z = 2.2 kΩ; cathode bypassed by C23 (100 nF).
  Drives only R_GA / R_GB (the two OPA454 summing-junction inputs) and
  the cathode-monitor's 1.5 V threshold divider on its own sheet
- Two OPA454 channels (U5 = Tube A, U10 = Tube B) each with R_F = 170 k,
  R_G = 10 k, R_GL = 22 k, R_pad = 1 k, plus 2N7000 bias-slam (Q2, Q3)
  sharing one R_GATE = 10 k. Transfer function V_out = 18·V_DAC - 85
- Shared bypass caps across U5/U10 V+ and V- rails (1 µF X7R bulk +
  100 nF HF on each rail); justified by grid-bias bandwidth being
  effectively DC vs textbook µV-class instrumentation recommendation

Supporting changes:

- New xmitter:OPA454 multi-unit symbol (Unit A = 3-pin op-amp triangle
  with IN-, IN+, OUT; Unit B = 5-pin power/enable block with V+, V-,
  ED, EDCOMM, STATFLG). Built via tools/add_opa454_symbol.py
- xmitter_prj/grid_bias.sch: V2 = 90 V (was 85), V3 = 5 V (was 12) to
  match the PDF design's +5 V / -90 V supply rails; LM4040 stays at 5 V
- pa_cathode_monitor.md: switch comparator V_REF from the bogus
  LM4040DIZ-1.2 (doesn't exist - LM4040 minimum is 2.048 V) to a shared
  LM4040DIZ-5.0 with a 4.7 k / 1 k trim / 1.5 k divider giving 1.5 V
  nominal (1.21 V to 1.74 V across full pot)
- Documentation/grid_bias.md: full subsystem design doc covering
  architecture decisions, transfer function, per-channel topology, BOM,
  inter-sheet I/O, calibration procedure, and open items
- Documentation/kicad_custom_symbols.md: OPA454 entry plus a note on
  the KiCad sub-symbol naming gotcha (NAME_{unit}_{body_style}, not th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
Changed lines of the file:
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@@
+	(wire
+		(pts
+			(xy 33.02 60.96) (xy 43.18 60.96)
+		)
+		(stroke
+			(width 0)
+			(type default)
+		)
+	)
 	(wire
 		(pts
@@
 	(hierarchical_label "3V3"
 		(shape output)
-		(at 43.18 60.96 180)
+		(at 33.02 60.96 180)
 		(effects
 			(font

Commit message: front-panel: QT encoder swap, PCF8575 breakout, pre-fab checklist, INT-none decision
Switch STEP + FUNC from direct PCF8575 GPIO to Adafruit I2C QT Rotary
Encoder breakouts (PID 4991) at addr 0x36 / 0x37. The onboard seesaw
SAMD09 handles quadrature decoding + button debounce, dropping ~200
lines of firmware. PCF8575 still covers the LCD (4-bit), paddle, and
panel LEDs.

Add custom KiCad symbols + footprints for both new breakouts to
xmitter.kicad_sym and xmitter.pretty. Footprint properties on the new
symbols are pre-linked, so schematic instances auto-associate. Some
coordinates in both footprints are best-guess pending physical
measurement -- flagged in the descr fields and in the new
front_panel_interface.md open-items subsections.

Decision documented (2026-07-03): no INT wiring back to the Metro.
Firmware polls all three I2C devices at 100 Hz; velocity-adaptive VFO
tuning is computed from delta-position / delta-time in the poll loop.
Rationale and a "here's how to add INT later" path in the new
"Interrupt handling (decision: none)" section of
front_panel_interface.md.

New Documentation/pcb_fab_checklist.md is the consolidated pre-flight
gate before analog-board gerbers ship -- nine sections covering
footprint verification, schematic completeness, ERC/DRC, physical, and
BOM sign-offs. build_checklist.md and CLAUDE.md updated to point at it.

Also in this bundle: SDA/SCL hierarchical labels changed to
bidirectional shape on the VFO, buffer_keyer, and interface sheets
(was an output/input polarity soup that would have failed ERC).
Interface and Front_Panel child sheets registered in .kicad_pro.
Front_Panel is an empty stub; components go in when the sheet is
populated. Adafruit PCF8575 and QT rotary encoder datasheets committed
under Documentation/Components/.

Co-Authored-By: Claude Opus 4.7 <noreply@anthropic.com>
Changed lines of the file:
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@@
 	)
 	(hierarchical_label "SDA"
-		(shape output)
+		(shape bidirectional)
 		(at 43.18 68.58 180)
 		(effects
@@
 	)
 	(hierarchical_label "SCL"
-		(shape output)
+		(shape bidirectional)
 		(at 43.18 66.04 180)
 		(effects

Commit message: schematic: I2C topology flip + CD14538B heartbeat + pre-layout audit
- Documentation updates for the STEMMA-QT topology flip (MCP4728 upstream
  of Si5351): design_review_7-5-26 C1 marked resolved, build_checklist
  Phase 1 gets the 6-step first-boot procedure, cw_envelope_keyer I2C
  address section rewritten, front_panel_interface signal-chain diagram
  refreshed.
- CD14538B dual retriggerable monostable added to xmitter.kicad_sym
  (PDIP-16, pinout verified against datasheet fig. 1), plus datasheet
  file.
- Arduino sheet: CD14538B heartbeat topology on Q5 HV contactor -- U18
  + R30 470K + C41 1uF timing (t_w ~470 ms), Q7 series FET stack,
  C42/C43 VDD bypass and bulk.
- Pre-layout audit output as Documentation/punch_list_7-6-26.txt (list
  of blockers before PCB layout, ordered by severity).

Co-Authored-By: Claude Opus 4.7 (1M context) <noreply@anthropic.com>
Parts:
- added TP1: RAW_RF, Connector_PinHeader_2.54mm:PinHeader_1x01_P2.54mm_Vertical, symbol Connector:TestPoint
Connections:
- net RAW_RF_OUT: now also TP1.1
- net SCL: no longer names the net of U1.SCL
- net SDA: no longer names the net of U1.SDA
- no-connect marks 0 -> 2
Changed lines of the file:
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@@
+	)
+	(junction
+		(at 213.36 66.04)
+		(diameter 0)
+		(color 0 0 0 0)
 	)
 	(junction
@@
 		(color 0 0 0 0)
 	)
+	(no_connect
+		(at 43.18 68.58)
+	)
+	(no_connect
+		(at 43.18 66.04)
+	)
 	(wire
 		(pts
@@
 	(wire
 		(pts
+			(xy 213.36 66.04) (xy 215.9 66.04)
+		)
+		(stroke
+			(width 0)
+			(type default)
+		)
+	)
+	(wire
+		(pts
 			(xy 104.14 62.23) (xy 116.84 62.23)
 		)
@@
 	(wire
 		(pts
-			(xy 204.47 66.04) (xy 215.9 66.04)
+			(xy 204.47 66.04) (xy 213.36 66.04)
 		)
 		(stroke
@@
 		)
 	)
-	(hierarchical_label "SDA"
-		(shape bidirectional)
-		(at 43.18 68.58 180)
-		(effects
-			(font
-				(size 1.27 1.27)
-			)
-			(justify right)
-		)
-	)
 	(hierarchical_label "RAW_RF_OUT"
 		(shape output)
@@
 			)
 			(justify left)
-		)
-	)
-	(hierarchical_label "SCL"
-		(shape bidirectional)
-		(at 43.18 66.04 180)
-		(effects
-			(font
-				(size 1.27 1.27)
-			)
-			(justify right)
 		)
 	)
@@
 					(unit 1)
 				)
+			)
+		)
+	)
+	(symbol
+		(lib_id "Connector:TestPoint")
+		(at 213.36 66.04 0)
+		(unit 1)
+		(body_style 1)
+		(exclude_from_sim no)
+		(in_bom yes)
+		(on_board yes)
+		(in_pos_files yes)
+		(dnp no)
+		(fields_autoplaced yes)
+		(property "Reference" "TP1"
+			(at 215.9 61.4679 0)
+			(show_name no)
+			(do_not_autoplace no)
+			(effects
+				(font
+					(size 1.27 1.27)
+				)
+				(justify left)
+			)
+		)
+		(property "Value" "RAW_RF"
+			(at 215.9 64.0079 0)
+			(show_name no)
+			(do_not_autoplace no)
+			(effects
+				(font
+					(size 1.27 1.27)
+				)
+				(justify left)
+			)
+		)
+		(property "Footprint" "Connector_PinHeader_2.54mm:PinHeader_1x01_P2.54mm_Vertical"
+			(at 218.44 66.04 0)
+			(hide yes)
+			(show_name no)
+			(do_not_autoplace no)
+			(effects
+				(font
+					(size 1.27 1.27)
+				)
+			)
+		)
+		(property "Datasheet" ""
+			(at 218.44 66.04 0)
+			(hide yes)
+			(show_name no)
+			(do_not_autoplace no)
+			(effects
+				(font
+					(size 1.27 1.27)
+				)
+			)
+		)
+		(property "Description" "test point"
+			(at 213.36 66.04 0)
+			(hide yes)
+			(show_name no)
+			(do_not_autoplace no)
+			(effects
+				(font
+					(size 1.27 1.27)
+				)
+			)
+		)
+		(pin "1"
+		)
+		(instances
+			(project "KiCAD"
+				(path "/d3de40b8-856b-4fbd-829c-f45ffcd55742/c08cbce4-6e06-48f3-b334-a48b1cc09989"
+					(reference "TP1")
+					(unit 1)
+				)
