File: KiCAD/vfo.kicad_sch (KiCad schematic)
At the start: 18 parts, among them Q1 J310, U1 Si5351A_Breakout

Commit message: kicad: convert hierarchical labels to globals (Path A) + unify _OUT/_IN pairs
- 58 hierarchical_label -> global_label conversions across the six active
  sheets. Standard KiCad 10 global_label form with fields_autoplaced +
  Intersheetrefs property.
- Stripped 36 vestigial sheet pins, 28 stitching wires, 2 junctions, 4
  labels from the root sheet. Sheet blocks remain; each is now a pure
  container with globals doing the cross-sheet connectivity by name.
- Renamed three OUT/IN pairs to unified names so same-name globals
  auto-connect:
    GRID_CTL_A_OUT + GRID_CTL_A_IN -> GRID_CTL_A
    GRID_CTL_B_OUT + GRID_CTL_B_IN -> GRID_CTL_B
    RAW_RF_OUT     + RAW_RF_IN     -> RAW_RF
- tools/convert_hier_to_global.py and tools/strip_root_stitching.py:
  reusable if we ever need to redo this.
- Documentation/punch_list_7-6-26.txt: mark B1a-e, L1, L2 resolved; add
  M6 (cosmetic) about GRID_CTL_A's label-at-pin-origin idiom; correct
  the earlier GRID_CTL_A false positive with the verified chain
  MCP4728 U8 VC -> R_PADA -> OPA454 U5 IN+ + Q3 drain.

Co-Authored-By: Claude Opus 4.7 (1M context) <noreply@anthropic.com>
Connections:
- net RAW_RF_OUT renamed RAW_RF
Changed lines of the file:
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@@
 		)
 	)
-	(hierarchical_label "3V3"
+	(global_label "3V3"
 		(shape output)
 		(at 33.02 60.96 180)
+		(fields_autoplaced yes)
 		(effects
 			(font
@@
 			(justify right)
 		)
+		(property "Intersheetrefs" "${INTERSHEET_REFS}"
+			(at 33.02 60.96 0)
+			(effects
+				(font
+					(size 1.27 1.27)
+				)
+				(hide yes)
+			)
+		)
 	)
-	(hierarchical_label "RAW_RF_OUT"
+	(global_label "RAW_RF"
 		(shape output)
 		(at 215.9 66.04 0)
+		(fields_autoplaced yes)
 		(effects
 			(font
@@
 			(justify left)
 		)
+		(property "Intersheetrefs" "${INTERSHEET_REFS}"
+			(at 215.9 66.04 0)
+			(effects
+				(font
+					(size 1.27 1.27)
+				)
+				(hide yes)
+			)
+		)
 	)

Commit message: kicad: PWR_FLAGs added, most +3.3V converted to 3V3, VFO renames + J2 NC
User work today:
- Placed PWR_FLAGs to silence "power_pin_not_driven" ERC errors for VEE,
  +12V, -90V rails (see B5a-B5f in the punch list)
- Converted 6 of 7 +3.3V power symbols to 3V3 global labels project-wide
  (one +3.3V remains on bias sheet, resolves next pass)
- VFO sheet: C_coup -> C_IN1, R6 -> RD1 (both were unannotated / duplicate
  ref designators; ERC B4a and B4b now resolved)
- buffer_keyer: J2 pin 2 gets a no_connect flag (B4c resolved); TP2 and
  TP7 electrically wired to MOD_RF_OUT+/- via junctions (B4d/e resolved)

Punch list updates:
- B3 (footprints) marked done
- B4a/b/c marked done
- M5 (TX LED) confirmed resolved (external LED across T/R relay coil)
- B2 (paddle) rewritten for the actual 2-conductor 1/4" plug scheme

Current ERC status: 61 errors, 0 warnings (from 74 + 2 originally).
Remaining real bugs: unannotated C_IN + duplicate C_IN1 on buffer_keyer,
misplaced #FLG04 on Metro's 3V3 pin, one leftover +3.3V on bias. Rest
are the known-non-issue plateau.

Co-Authored-By: Claude Opus 4.7 (1M context) <noreply@anthropic.com>
Parts:
- renumbered C_coup to C_IN1, R6 to RD1, RS to RS1
Connections:
- no-connect marks 2 -> 4
Changed lines of the file:
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@@
 		(at 43.18 66.04)
+	)
+	(no_connect
+		(at 58.42 67.31)
+	)
+	(no_connect
+		(at 58.42 64.77)
 	)
 	(wire
@@
 		(dnp no)
 		(fields_autoplaced yes)
-		(property "Reference" "RS"
+		(property "Reference" "RS1"
 			(at 72.3899 59.69 0)
 			(show_name no)
@@
 			(project "KiCAD"
 				(path "/d3de40b8-856b-4fbd-829c-f45ffcd55742/c08cbce4-6e06-48f3-b334-a48b1cc09989"
-					(reference "RS")
+					(reference "RS1")
 					(unit 1)
 				)
@@
 		(dnp no)
 		(fields_autoplaced yes)
-		(property "Reference" "R6"
+		(property "Reference" "RD1"
 			(at 207.01 68.5799 0)
 			(show_name no)
@@
 			(project "KiCAD"
 				(path "/d3de40b8-856b-4fbd-829c-f45ffcd55742/c08cbce4-6e06-48f3-b334-a48b1cc09989"
-					(reference "R6")
+					(reference "RD1")
 					(unit 1)
 				)
@@
 		(dnp no)
 		(fields_autoplaced yes)
-		(property "Reference" "C_coup"
+		(property "Reference" "C_IN1"
 			(at 86.36 54.61 90)
 			(show_name no)
@@
 			(project "KiCAD"
 				(path "/d3de40b8-856b-4fbd-829c-f45ffcd55742/c08cbce4-6e06-48f3-b334-a48b1cc09989"
-					(reference "C_coup")
+					(reference "C_IN1")
 					(unit 1)
 				)

Commit message: kicad: VFO placed on PCB; Si5351 STEMMA footprint rebuilt
- Adafruit_Si5351A_STEMMA.kicad_mod: rebuilt from physical breakout as
  2-row 10-pad through-hole with GND spacers between clocks. Top row:
  CLK2/GND/CLK1/GND/CLK0; bottom row: VIN/(NC)/GND/SCL/SDA. Mounting-hole
  rectangle 20.32 x 12.70 mm; pin rows at Y=+/-6.35 mm.
- vfo.kicad_sch: removed CLK2 no_connect so VFO can source from CLK2
  (shorter physical trace than CLK0). CLK0/CLK1/SDA/SCL still NC.
- KiCAD.kicad_pcb: initial VFO component placement on 200x150 mm board.
  Toroids L2/L4/L6 spaced 40/46 mm c-c (~23/29 mm edge-edge) so vertical
  L4 mount is no longer required. C44 100 nF within ~6 mm of Q1.
- build_checklist.md: pre-assembly verify for U11 LM4040 (LP-5 has pin 1
  = NC, some package variants map A/K differently).
- tools/vfo_placement_audit.py: repeatable placement audit (board-fit,
  toroid spacing, signal chain, via count, CLK0-vs-CLK2 comparison).
- .gitignore: KiCad generated reports (ERC.rpt, report.txt, DRC.rpt).

Co-Authored-By: Claude Opus 4.7 <noreply@anthropic.com>
Parts:
- added C44: 100nF, Capacitor_THT:C_Disc_D5.0mm_W2.5mm_P5.00mm, symbol Device:C
Connections:
- net +12V: now also C44.1
- net GND: now also C44.2
- net at RS1.1: now also U1.CLK2; no longer U1.CLK0
Other:
- moved on the sheet: U1

Commit message: kicad: T68-6 hand-wound toroid footprints (flat + vertical)
- xmitter.pretty/T68-6_Flat_HandWound.kicad_mod: flat mount for L2/L6.
  Both leads exit on the same radial side -- outer pad at (0, -10.0)
  1.23 mm outside OD, inner pad at (0, -2.5) inside the ID hole.
  Pitch 7.5 mm. Silk shows OD (17.53 mm) + ID (9.40 mm) circles.
- xmitter.pretty/T68-6_Vertical_HandWound.kicad_mod: on-edge mount for L4.
  Top-down projection = OD x HT (17.53 x 4.83 mm) rectangle. Pads at
  (-2.0, -4.5) and (+2.0, +4.5) -- above and below the rectangle with
  the diagonal offset that matches natural lead exit after 4-turn winding.
- vfo.kicad_sch: L2/L4/L6 footprint fields switched to the new project
  footprints (was Inductor_THT:L_Toroid_Horizontal_D17.3mm_P15.24mm_Bourns_2000
  which is a pre-wound Bourns part, not a hand-wound toroid).
- Documentation/flat-toroid.jpg: reference drawing showing lead
  arrangement for both mount styles.

Nominal L per inductor with 4 turns of 22/24 AWG magnet wire evenly
spaced: A_L(T68-6) * 4^2 = 47 * 16 = 752 nH (target 736 nH, +2.2%).

Co-Authored-By: Claude Opus 4.7 <noreply@anthropic.com>
Parts:
- L2, L6: footprint Inductor_THT:L_Toroid_Horizontal_D17.3mm_P15.24mm_Bourns_2000 -> xmitter:T68-6_Flat_HandWound
- L4: footprint Inductor_THT:L_Toroid_Horizontal_D17.3mm_P15.24mm_Bourns_2000 -> xmitter:T68-6_Vertical_HandWound
Changed lines of the file:
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@@
 			)
 		)
-		(property "Footprint" "Inductor_THT:L_Toroid_Horizontal_D17.3mm_P15.24mm_Bourns_2000"
+		(property "Footprint" "xmitter:T68-6_Flat_HandWound"
 			(at 163.83 62.23 0)
 			(hide yes)
@@
 			)
 		)
-		(property "Footprint" "Inductor_THT:L_Toroid_Horizontal_D17.3mm_P15.24mm_Bourns_2000"
+		(property "Footprint" "xmitter:T68-6_Vertical_HandWound"
 			(at 142.24 62.23 0)
 			(hide yes)
@@
 			)
 		)
-		(property "Footprint" "Inductor_THT:L_Toroid_Horizontal_D17.3mm_P15.24mm_Bourns_2000"
+		(property "Footprint" "xmitter:T68-6_Flat_HandWound"
 			(at 120.65 62.23 0)
 			(hide yes)

Commit message: kicad: fix L7 to Device:L symbol, add JFET gate leak on VFO
- buffer_keyer.kicad_sch: L7 (22uH choke) now uses Device:L symbol
  instead of Device:R. Netlist and footprint unchanged; symbol now
  renders as inductor loops instead of resistor rectangle.
- vfo.kicad_sch + PCB: added 10K gate-leak resistor at Q1 (J310 buffer)
  to provide DC gate reference. Was missing from KiCad implementation
  but present in QUCS reference schematic as RGL 1M (10K is fine).
- 5 initial mounting holes placed on PCB (positions will be reworked in
  the next commit).

Co-Authored-By: Claude Opus 4.7 <noreply@anthropic.com>
Parts:
- added R17: 10K, Resistor_THT:R_Axial_DIN0207_L6.3mm_D2.5mm_P10.16mm_Horizontal, symbol Device:R_US
Connections:
- net GND: now also R17.2
- net at CC1.2, Q1.2 (G): now also R17.1
Changed lines of the file:
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@@
+	)
+	(junction
+		(at 195.58 62.23)
+		(diameter 0)
+		(color 0 0 0 0)
 	)
 	(junction
@@
 	(wire
 		(pts
-			(xy 204.47 55.88) (xy 204.47 57.15)
+			(xy 195.58 62.23) (xy 196.85 62.23)
 		)
 		(stroke
@@
 	(wire
 		(pts
-			(xy 204.47 66.04) (xy 204.47 67.31)
+			(xy 204.47 55.88) (xy 204.47 57.15)
 		)
 		(stroke
@@
 	(wire
 		(pts
-			(xy 132.08 62.23) (xy 138.43 62.23)
+			(xy 204.47 66.04) (xy 204.47 67.31)
 		)
 		(stroke
@@
 	(wire
 		(pts
-			(xy 90.17 62.23) (xy 95.25 62.23)
+			(xy 132.08 62.23) (xy 138.43 62.23)
 		)
 		(stroke
@@
 	(wire
 		(pts
-			(xy 104.14 63.5) (xy 104.14 62.23)
+			(xy 90.17 62.23) (xy 95.25 62.23)
 		)
 		(stroke
@@
 	(wire
 		(pts
-			(xy 180.34 62.23) (xy 185.42 62.23)
+			(xy 104.14 63.5) (xy 104.14 62.23)
 		)
 		(stroke
@@
 	(wire
 		(pts
-			(xy 58.42 62.23) (xy 69.85 62.23)
+			(xy 180.34 62.23) (xy 185.42 62.23)
 		)
 		(stroke
@@
 	(wire
 		(pts
-			(xy 193.04 62.23) (xy 196.85 62.23)
+			(xy 58.42 62.23) (xy 69.85 62.23)
+		)
+		(stroke
+			(width 0)
+			(type default)
+		)
+	)
+	(wire
+		(pts
+			(xy 193.04 62.23) (xy 195.58 62.23)
 		)
 		(stroke
@@
 				(path "/d3de40b8-856b-4fbd-829c-f45ffcd55742/c08cbce4-6e06-48f3-b334-a48b1cc09989"
 					(reference "#PWR03")
+					(unit 1)
+				)
+			)
+		)
+	)
+	(symbol
+		(lib_id "Device:R_US")
+		(at 195.58 66.04 0)
+		(unit 1)
+		(body_style 1)
+		(exclude_from_sim no)
+		(in_bom yes)
+		(on_board yes)
+		(in_pos_files yes)
+		(dnp no)
+		(fields_autoplaced yes)
+		(property "Reference" "R17"
+			(at 198.12 64.7699 0)
+			(show_name no)
+			(do_not_autoplace no)
+			(effects
+				(font
+					(size 1.27 1.27)
+				)
+				(justify left)
+			)
+		)
+		(property "Value" "10K"
+			(at 198.12 67.3099 0)
+			(show_name no)
+			(do_not_autoplace no)
+			(effects
+				(font
+					(size 1.27 1.27)
+				)
+				(justify left)
+			)
+		)
+		(property "Footprint" "Resistor_THT:R_Axial_DIN0207_L6.3mm_D2.5mm_P10.16mm_Horizontal"
+			(at 196.596 66.294 90)
+			(hide yes)
+			(show_name no)
+			(do_not_autoplace no)
+			(effects
+				(font
+					(size 1.27 1.27)
+				)
+			)
+		)
+		(property "Datasheet" ""
+			(at 195.58 66.04 0)
+			(hide yes)
+			(show_name no)
+			(do_not_autoplace no)
+			(effects
+				(font
+					(size 1.27 1.27)
+				)
+			)
+		)
+		(property "Description" "Resistor, US symbol"
+			(at 195.58 66.04 0)
+			(hide yes)
+			(show_name no)
+			(do_not_autoplace no)
+			(effects
+				(font
+					(size 1.27 1.27)
+				)
+			)
+		)
+		(pin "2"
+		)
+		(pin "1"
+		)
+		(instances
+			(project "KiCAD"
+				(path "/d3de40b8-856b-4fbd-829c-f45ffcd55742/c08cbce4-6e06-48f3-b334-a48b1cc09989"
+					(reference "R17")
 					(unit 1)
 				)
@@
 					(unit 1)
 				)
+			)
+		)
+	)
+	(symbol
+		(lib_id "power:GND")
+		(at 195.58 69.85 0)
+		(unit 1)
+		(body_style 1)
+		(exclude_from_sim no)
+		(in_bom yes)
+		(on_board yes)
+		(in_pos_files yes)
+		(dnp no)
+		(fields_autoplaced yes)
+		(property "Reference" "#PWR055"
+			(at 195.58 76.2 0)
+			(hide yes)
+			(show_name no)
+			(do_not_autoplace no)
+			(effects
+				(font
+					(size 1.27 1.27)
+				)
+			)
+		)
+		(property "Value" "GND"
+			(at 195.58 74.93 0)
+			(show_name no)
+			(do_not_autoplace no)
+			(effects
+				(font
+					(size 1.27 1.27)
+				)
+			)
+		)
+		(property "Footprint" ""
+			(at 195.58 69.85 0)
+			(hide yes)
+			(show_name no)
+			(do_not_autoplace no)
+			(effects
+				(font
+					(size 1.27 1.27)
+				)
+			)
+		)
+		(property "Datasheet" ""
+			(at 195.58 69.85 0)
+			(hide yes)
+			(show_name no)
+			(do_not_autoplace no)
+			(effects
+				(font
+					(size 1.27 1.27)
+				)
+			)
+		)
+		(property "Description" "Power symbol creates a global label with name \"GND\" , ground"
+			(at 195.58 69.85 0)
+			(hide yes)
+			(show_name no)
+			(do_not_autoplace no)
+			(effects
+				(font
+					(size 1.27 1.27)
+				)
+			)
+		)
+		(pin "1"
+		)
+		(instances
+			(project "KiCAD"
+				(path "/d3de40b8-856b-4fbd-829c-f45ffcd55742/c08cbce4-6e06-48f3-b334-a48b1cc09989"
+					(reference "#PWR055")
+					(unit 1)
+				)
