File: KiCAD/interface.kicad_sch (KiCad schematic)
At the start: 11 parts, among them J15 Conn_01x03_Pin, J4 8P8C_Shielded, U16 AM26LS32ACN

Commit message: kicad: convert hierarchical labels to globals (Path A) + unify _OUT/_IN pairs
- 58 hierarchical_label -> global_label conversions across the six active
  sheets. Standard KiCad 10 global_label form with fields_autoplaced +
  Intersheetrefs property.
- Stripped 36 vestigial sheet pins, 28 stitching wires, 2 junctions, 4
  labels from the root sheet. Sheet blocks remain; each is now a pure
  container with globals doing the cross-sheet connectivity by name.
- Renamed three OUT/IN pairs to unified names so same-name globals
  auto-connect:
    GRID_CTL_A_OUT + GRID_CTL_A_IN -> GRID_CTL_A
    GRID_CTL_B_OUT + GRID_CTL_B_IN -> GRID_CTL_B
    RAW_RF_OUT     + RAW_RF_IN     -> RAW_RF
- tools/convert_hier_to_global.py and tools/strip_root_stitching.py:
  reusable if we ever need to redo this.
- Documentation/punch_list_7-6-26.txt: mark B1a-e, L1, L2 resolved; add
  M6 (cosmetic) about GRID_CTL_A's label-at-pin-origin idiom; correct
  the earlier GRID_CTL_A false positive with the verified chain
  MCP4728 U8 VC -> R_PADA -> OPA454 U5 IN+ + Q3 drain.

Co-Authored-By: Claude Opus 4.7 (1M context) <noreply@anthropic.com>
Changed lines of the file:
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@@
 		)
 	)
-	(hierarchical_label "MBL_B_P"
+	(global_label "MBL_B_P"
 		(shape output)
 		(at 109.22 97.79 180)
-		(effects
-			(font
-				(size 1.27 1.27)
-			)
-			(justify right)
-		)
-	)
-	(hierarchical_label "MBL_A_P"
+		(fields_autoplaced yes)
+		(effects
+			(font
+				(size 1.27 1.27)
+			)
+			(justify right)
+		)
+		(property "Intersheetrefs" "${INTERSHEET_REFS}"
+			(at 109.22 97.79 0)
+			(effects
+				(font
+					(size 1.27 1.27)
+				)
+				(hide yes)
+			)
+		)
+	)
+	(global_label "MBL_A_P"
 		(shape output)
 		(at 109.22 92.71 180)
-		(effects
-			(font
-				(size 1.27 1.27)
-			)
-			(justify right)
-		)
-	)
-	(hierarchical_label "SDA"
+		(fields_autoplaced yes)
+		(effects
+			(font
+				(size 1.27 1.27)
+			)
+			(justify right)
+		)
+		(property "Intersheetrefs" "${INTERSHEET_REFS}"
+			(at 109.22 92.71 0)
+			(effects
+				(font
+					(size 1.27 1.27)
+				)
+				(hide yes)
+			)
+		)
+	)
+	(global_label "SDA"
 		(shape bidirectional)
 		(at 35.56 101.6 0)
-		(effects
-			(font
-				(size 1.27 1.27)
-			)
-			(justify left)
-		)
-	)
-	(hierarchical_label "SCL"
+		(fields_autoplaced yes)
+		(effects
+			(font
+				(size 1.27 1.27)
+			)
+			(justify left)
+		)
+		(property "Intersheetrefs" "${INTERSHEET_REFS}"
+			(at 35.56 101.6 0)
+			(effects
+				(font
+					(size 1.27 1.27)
+				)
+				(hide yes)
+			)
+		)
+	)
+	(global_label "SCL"
 		(shape bidirectional)
 		(at 35.56 99.06 0)
-		(effects
-			(font
-				(size 1.27 1.27)
-			)
-			(justify left)
-		)
-	)
-	(hierarchical_label "MBL_A_P"
+		(fields_autoplaced yes)
+		(effects
+			(font
+				(size 1.27 1.27)
+			)
+			(justify left)
+		)
+		(property "Intersheetrefs" "${INTERSHEET_REFS}"
+			(at 35.56 99.06 0)
+			(effects
+				(font
+					(size 1.27 1.27)
+				)
+				(hide yes)
+			)
+		)
+	)
+	(global_label "MBL_A_P"
 		(shape output)
 		(at 54.61 135.89 180)
-		(effects
-			(font
-				(size 1.27 1.27)
-			)
-			(justify right)
-		)
-	)
-	(hierarchical_label "MBL_A_N"
+		(fields_autoplaced yes)
+		(effects
+			(font
+				(size 1.27 1.27)
+			)
+			(justify right)
+		)
+		(property "Intersheetrefs" "${INTERSHEET_REFS}"
+			(at 54.61 135.89 0)
+			(effects
+				(font
+					(size 1.27 1.27)
+				)
+				(hide yes)
+			)
+		)
+	)
+	(global_label "MBL_A_N"
 		(shape output)
 		(at 77.47 128.27 180)
-		(effects
-			(font
-				(size 1.27 1.27)
-			)
-			(justify right)
-		)
-	)
-	(hierarchical_label "MBL_B_P"
+		(fields_autoplaced yes)
+		(effects
+			(font
+				(size 1.27 1.27)
+			)
+			(justify right)
+		)
+		(property "Intersheetrefs" "${INTERSHEET_REFS}"
+			(at 77.47 128.27 0)
+			(effects
+				(font
+					(size 1.27 1.27)
+				)
+				(hide yes)
+			)
+		)
+	)
+	(global_label "MBL_B_P"
 		(shape output)
 		(at 58.42 71.12 180)
-		(effects
-			(font
-				(size 1.27 1.27)
-			)
-			(justify right)
-		)
-	)
-	(hierarchical_label "MBL_B_N"
+		(fields_autoplaced yes)
+		(effects
+			(font
+				(size 1.27 1.27)
+			)
+			(justify right)
+		)
+		(property "Intersheetrefs" "${INTERSHEET_REFS}"
+			(at 58.42 71.12 0)
+			(effects
+				(font
+					(size 1.27 1.27)
+				)
+				(hide yes)
+			)
+		)
+	)
+	(global_label "MBL_B_N"
 		(shape output)
 		(at 74.93 78.74 180)
-		(effects
-			(font
-				(size 1.27 1.27)
-			)
-			(justify right)
-		)
-	)
-	(hierarchical_label "MBL_A_N"
+		(fields_autoplaced yes)
+		(effects
+			(font
+				(size 1.27 1.27)
+			)
+			(justify right)
+		)
+		(property "Intersheetrefs" "${INTERSHEET_REFS}"
+			(at 74.93 78.74 0)
+			(effects
+				(font
+					(size 1.27 1.27)
+				)
+				(hide yes)
+			)
+		)
+	)
+	(global_label "MBL_A_N"
 		(shape output)
 		(at 109.22 95.25 180)
-		(effects
-			(font
-				(size 1.27 1.27)
-			)
-			(justify right)
-		)
-	)
-	(hierarchical_label "MBL600_B"
+		(fields_autoplaced yes)
+		(effects
+			(font
+				(size 1.27 1.27)
+			)
+			(justify right)
+		)
+		(property "Intersheetrefs" "${INTERSHEET_REFS}"
+			(at 109.22 95.25 0)
+			(effects
+				(font
+					(size 1.27 1.27)
+				)
+				(hide yes)
+			)
+		)
+	)
+	(global_label "MBL600_B"
 		(shape output)
 		(at 153.67 97.79 0)
-		(effects
-			(font
-				(size 1.27 1.27)
-			)
-			(justify left)
-		)
-	)
-	(hierarchical_label "MBL_B_N"
+		(fields_autoplaced yes)
+		(effects
+			(font
+				(size 1.27 1.27)
+			)
+			(justify left)
+		)
+		(property "Intersheetrefs" "${INTERSHEET_REFS}"
+			(at 153.67 97.79 0)
+			(effects
+				(font
+					(size 1.27 1.27)
+				)
+				(hide yes)
+			)
+		)
+	)
+	(global_label "MBL_B_N"
 		(shape output)
 		(at 109.22 100.33 180)
-		(effects
-			(font
-				(size 1.27 1.27)
-			)
-			(justify right)
-		)
-	)
-	(hierarchical_label "MBL600_A"
+		(fields_autoplaced yes)
+		(effects
+			(font
+				(size 1.27 1.27)
+			)
+			(justify right)
+		)
+		(property "Intersheetrefs" "${INTERSHEET_REFS}"
+			(at 109.22 100.33 0)
+			(effects
+				(font
+					(size 1.27 1.27)
+				)
+				(hide yes)
+			)
+		)
+	)
+	(global_label "MBL600_A"
 		(shape output)
 		(at 173.99 92.71 0)
-		(effects
-			(font
-				(size 1.27 1.27)
-			)
-			(justify left)
-		)
-	)
+		(fields_autoplaced yes)
+		(effects
+			(font
+				(size 1.27 1.27)
+			)
+			(justify left)
+		)
+		(property "Intersheetrefs" "${INTERSHEET_REFS}"
+			(at 173.99 92.71 0)
+			(effects
+				(font
+					(size 1.27 1.27)
+				)
+				(hide yes)
+			)
+		)
+	)

Commit message: kicad: fill 9 remaining footprints across active sheets
- arduino: R30 470K (R_Axial_DIN0207 horizontal), C41 1uF (rect L7.2mm),
  C42 100nF (disc D5mm P5mm), C43 10uF (radial polarized D5mm P2mm)
- bias: J11 (GRID_BIAS), J12 (CATHODE_SENSE), J14 -- all PinHeader_1x02
  vertical THT
- buffer_keyer: J13 -- PinHeader_1x05 vertical THT
- interface: J15 -- PinHeader_1x03 vertical THT

C41/C42/C43 filled by re-running tools/assign_cap_footprints.py which
already had the intended mappings. R30 and the connectors done by hand
via a one-off script.

Only U2 (Metro) remains footprint-less, intentionally off-PCB.

Punch list updates for today's ERC pass + user's schematic edits:
- B3 (footprints) resolved.
- B4d/B4e (TP2/TP7 to MOD_RF+/-) resolved -- user verified junction dots
  + wires in KiCad. TP3 = SCL is intentional (I2C debug probe access).
- M5 (TX_LED) previously resolved -- LED wired in parallel with T/R
  relay coil, no Metro GPIO needed.
- B2 (paddle) rewritten for the actual design: J10 = 2-conductor 1/4"
  phone plug, tip -> Metro D5, sleeve -> GND.

vfo.kicad_sch diff is KiCad's own canonicalization of Intersheetrefs
property (show_name/do_not_autoplace fields shuffled) from opening +
saving; contents equivalent.

Co-Authored-By: Claude Opus 4.7 (1M context) <noreply@anthropic.com>
Parts:
- J15: footprint (none) -> Connector_PinHeader_2.54mm:PinHeader_1x03_P2.54mm_Vertical
Changed lines of the file:
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@@
 		(property "Intersheetrefs" "${INTERSHEET_REFS}"
 			(at 109.22 97.79 0)
-			(effects
-				(font
-					(size 1.27 1.27)
-				)
-				(hide yes)
+			(hide yes)
+			(show_name no)
+			(do_not_autoplace no)
+			(effects
+				(font
+					(size 1.27 1.27)
+				)
 			)
 		)
@@
 		(property "Intersheetrefs" "${INTERSHEET_REFS}"
 			(at 109.22 92.71 0)
-			(effects
-				(font
-					(size 1.27 1.27)
-				)
-				(hide yes)
+			(hide yes)
+			(show_name no)
+			(do_not_autoplace no)
+			(effects
+				(font
+					(size 1.27 1.27)
+				)
 			)
 		)
@@
 		(property "Intersheetrefs" "${INTERSHEET_REFS}"
 			(at 35.56 101.6 0)
-			(effects
-				(font
-					(size 1.27 1.27)
-				)
-				(hide yes)
+			(hide yes)
+			(show_name no)
+			(do_not_autoplace no)
+			(effects
+				(font
+					(size 1.27 1.27)
+				)
 			)
 		)
@@
 		(property "Intersheetrefs" "${INTERSHEET_REFS}"
 			(at 35.56 99.06 0)
-			(effects
-				(font
-					(size 1.27 1.27)
-				)
-				(hide yes)
+			(hide yes)
+			(show_name no)
+			(do_not_autoplace no)
+			(effects
+				(font
+					(size 1.27 1.27)
+				)
 			)
 		)
@@
 		(property "Intersheetrefs" "${INTERSHEET_REFS}"
 			(at 54.61 135.89 0)
-			(effects
-				(font
-					(size 1.27 1.27)
-				)
-				(hide yes)
+			(hide yes)
+			(show_name no)
+			(do_not_autoplace no)
+			(effects
+				(font
+					(size 1.27 1.27)
+				)
 			)
 		)
@@
 		(property "Intersheetrefs" "${INTERSHEET_REFS}"
 			(at 77.47 128.27 0)
-			(effects
-				(font
-					(size 1.27 1.27)
-				)
-				(hide yes)
+			(hide yes)
+			(show_name no)
+			(do_not_autoplace no)
+			(effects
+				(font
+					(size 1.27 1.27)
+				)
 			)
 		)
@@
 		(property "Intersheetrefs" "${INTERSHEET_REFS}"
 			(at 58.42 71.12 0)
-			(effects
-				(font
-					(size 1.27 1.27)
-				)
-				(hide yes)
+			(hide yes)
+			(show_name no)
+			(do_not_autoplace no)
+			(effects
+				(font
+					(size 1.27 1.27)
+				)
 			)
 		)
@@
 		(property "Intersheetrefs" "${INTERSHEET_REFS}"
 			(at 74.93 78.74 0)
-			(effects
-				(font
-					(size 1.27 1.27)
-				)
-				(hide yes)
+			(hide yes)
+			(show_name no)
+			(do_not_autoplace no)
+			(effects
+				(font
+					(size 1.27 1.27)
+				)
 			)
 		)
@@
 		(property "Intersheetrefs" "${INTERSHEET_REFS}"
 			(at 109.22 95.25 0)
-			(effects
-				(font
-					(size 1.27 1.27)
-				)
-				(hide yes)
+			(hide yes)
+			(show_name no)
+			(do_not_autoplace no)
+			(effects
+				(font
+					(size 1.27 1.27)
+				)
 			)
 		)
@@
 		(property "Intersheetrefs" "${INTERSHEET_REFS}"
 			(at 153.67 97.79 0)
-			(effects
-				(font
-					(size 1.27 1.27)
-				)
-				(hide yes)
+			(hide yes)
+			(show_name no)
+			(do_not_autoplace no)
+			(effects
+				(font
+					(size 1.27 1.27)
+				)
 			)
 		)
@@
 		(property "Intersheetrefs" "${INTERSHEET_REFS}"
 			(at 109.22 100.33 0)
-			(effects
-				(font
-					(size 1.27 1.27)
-				)
-				(hide yes)
+			(hide yes)
+			(show_name no)
+			(do_not_autoplace no)
+			(effects
+				(font
+					(size 1.27 1.27)
+				)
 			)
 		)
@@
 		(property "Intersheetrefs" "${INTERSHEET_REFS}"
 			(at 173.99 92.71 0)
-			(effects
-				(font
-					(size 1.27 1.27)
-				)
-				(hide yes)
+			(hide yes)
+			(show_name no)
+			(do_not_autoplace no)
+			(effects
+				(font
+					(size 1.27 1.27)
+				)
 			)
 		)
@@
 			)
 		)
-		(property "Footprint" ""
+		(property "Footprint" "Connector_PinHeader_2.54mm:PinHeader_1x03_P2.54mm_Vertical"
 			(at 175.26 105.41 0)
 			(hide yes)
