File: KiCAD/frontpanel/frontpanel.kicad_pcb (KiCad board)
At the start: 2 copper layers, 27 parts, among them J1 8P8C_Shielded, Q1 2N7000, Q2 2N7000, Q3 2N7000, U1 Adafruit_PCF8575_Breakout, U2 MCP4725

Commit message: Front-panel PCB: layout complete, DFM verified, ready for fab
Complete the front-panel PCB layout.  ERC clean, DRC clean except for
two silk_over_copper warnings on J1 SH pads (cosmetic; RJE1D-188
footprint silk box crosses the shield tab pads.  Irrelevant since the
shield is intentionally left floating on this board).

Layout details:

  - Board: 78 x 85 mm, 4x M3 corner mounting holes at 4 mm inset.
  - GND pours on F.Cu and B.Cu.  RJ45 shield isolation keepout
    (17.5 x 16 mm) on both layers prevents pour from touching the
    floating SH tabs.
  - Track widths 0.2 - 0.5 mm (JLC min 0.127 mm).  4 vias, 142 tracks.
  - Drill sizes 0.3 - 3.0 mm (JLC min 0.3 mm; aspect ratio 5.3:1 max
    on the 1.6 mm board).
  - J2 (Conn_01x03_Pin) added to bring out PCF8575 P13/P14/P15 for
    future use.  TP9 GND test point added.
  - PCF8575 P0-P3 also routed to LCD DB0-DB3: physically wired but
    ignored in 4-bit mode.  Per-pin jumpers at the LCD header let
    the trace be dropped if P0-P3 need reallocation.  8-bit mode
    is a firmware-only upgrade.
  - TP3 / TP4 value fields cleaned up (BLUE+IN -> BLUE_IN,
    GREEN__IN -> GREEN_IN).

Fix xmitter:Amphenol_RJE1D-188_Horizontal_Shielded footprint: previous
version had all Y coordinates negated relative to the PCB edge, which
caused the connector to sit backwards when placed.  Reworked to put
PCB edge below origin at Y=+8.8 and pin block above at Y=-3.96 /
Y=-6.50, matching the datasheet.

Docs:
  - front_panel_interface.md: full PCF8575 -> LCD pin allocation
    table, noting that P0-P3 are wired-but-ignored in 4-bit mode.
  - kicad_routing_cheatsheet.md: "B doesn't fill my pour"
    troubleshooting section (5 causes ordered by frequency).

Co-Authored-By: Claude Opus 4.7 <noreply@anthropic.com>
Parts:
- added J2: Conn_01x03_Pin, Connector_PinHeader_2.54mm:PinHeader_1x03_P2.54mm_Vertical, F.Cu at (135.3, 104.0)
- added TP9: GND, Connector_PinHeader_2.54mm:PinHeader_1x01_P2.54mm_Vertical, F.Cu at (135.0, 99.6)
- TP3: value BLUE+IN -> BLUE_IN
- TP4: value GREEN__IN -> GREEN_IN
- moved LCD1 275.8 mm to (172.7, 119.2), turned to 180 degrees
- moved C4 258.7 mm to (167.1, 115.5), turned to -90 degrees
- moved R3 252.8 mm to (167.6, 64.1), turned to 90 degrees
- moved R2 244.6 mm to (159.8, 64.0), turned to 90 degrees
- moved C12 241.6 mm to (150.0, 122.8)
- moved R1 236.4 mm to (152.1, 63.9), turned to 90 degrees
- moved C3 231.1 mm to (167.3, 107.6), turned to -90 degrees
- moved U1 228.1 mm to (153.9, 98.0), turned to 90 degrees
- moved C11 223.1 mm to (159.0, 122.9)
- moved C6 222.6 mm to (131.8, 96.6), turned to 180 degrees
- moved C2 216.3 mm to (125.1, 104.7)
- moved Q3 215.0 mm to (167.6, 68.4), turned to -90 degrees
- moved TP5 214.5 mm to (167.4, 75.4), turned to 180 degrees
- moved TP6 214.3 mm to (167.4, 81.5), turned to 180 degrees
- moved TP7 209.2 mm to (167.4, 87.2), turned to 180 degrees
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Connections:
- LCD1 pad 10: unconnected-(LCD1-DB3-Pad10) -> /LCD_D3
- LCD1 pad 7: unconnected-(LCD1-DB0-Pad7) -> /LCD_D0
- LCD1 pad 8: unconnected-(LCD1-DB1-Pad8) -> /LCD_D1
- LCD1 pad 9: unconnected-(LCD1-DB2-Pad9) -> /LCD_D2
- U1 pad P0: unconnected-(U1-PadP0) -> /LCD_D0
- U1 pad P1: unconnected-(U1-PadP1) -> /LCD_D1
- U1 pad P13: unconnected-(U1-PadP13) -> Net-(J2-Pin_1)
- U1 pad P14: unconnected-(U1-PadP14) -> Net-(J2-Pin_2)
- U1 pad P15: unconnected-(U1-PadP15) -> Net-(J2-Pin_3)
- U1 pad P2: unconnected-(U1-PadP2) -> /LCD_D2
- U1 pad P3: unconnected-(U1-PadP3) -> /LCD_D3
Routing:
- net +5V: track 0.00 -> 200.2 mm
- net SDA: track 0.00 -> 76.8 mm
- net SCL: track 0.00 -> 70.6 mm
- net Net-(LCD1-V0): track 0.00 -> 67.2 mm
- net Net-(LCD1-E): track 0.00 -> 42.5 mm
- net Net-(LCD1-R): track 0.00 -> 39.2 mm
- net BLUE: track 0.00 -> 38.5 mm, vias 0 -> 1
- net Net-(LCD1-RS): track 0.00 -> 32.5 mm
- net GREEN: track 0.00 -> 31.5 mm, vias 0 -> 1
- net RED: track 0.00 -> 27.4 mm
- net Net-(LCD1-G): track 0.00 -> 20.4 mm
- net Net-(J2-Pin_1): track 0.00 -> 15.3 mm
- net /LCD_D0: track 0.00 -> 14.6 mm, vias 0 -> 1
- net /LCD_D3: track 0.00 -> 13.5 mm
- net /LCD_D7: track 0.00 -> 13.3 mm
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- added copper zone on B.Cu, net GND
- added copper zone on F.Cu, net GND
Other:
- board outline added: 78 x 85 mm
- board text added: "Front Panel Rev A"

Commit message: Front-panel PCB: re-add corner mounting holes; ignore fab outputs
Re-add four M3 corner mounting holes (MH1-MH4 at 4 mm inset from the
78 x 85 mm board edges) that got wiped when the layout was redone.
Same specs as the analog board: MountingHole:MountingHole_3.2mm_M3,
non-plated Ø3.2 mm.  Chassis-side mounting scheme; the courtyard-
overlap warning between MH3 and U2 is a DRC false-alarm for this
board (no top-side hardware).

Also extend .gitignore to cover:
  - Gerber output directories and archives (regenerable from
    .kicad_pcb; standard convention for KiCad projects).
  - ERC/DRC/report files in per-board subdirectories (previously
    only the top-level ones were ignored).

Front-panel Rev A gerbers submitted to JLCPCB 2026-07-20; the
frontpanel.kicad_pcb at this commit is the fab-order source.

Co-Authored-By: Claude Opus 4.7 <noreply@anthropic.com>
Parts:
- added MH1: MountingHole_3.2mm_M3, MountingHole:MountingHole_3.2mm_M3, F.Cu at (104.5, 52.5)
- added MH2: MountingHole_3.2mm_M3, MountingHole:MountingHole_3.2mm_M3, F.Cu at (174.5, 52.5)
- added MH3: MountingHole_3.2mm_M3, MountingHole:MountingHole_3.2mm_M3, F.Cu at (104.5, 129.5)
- added MH4: MountingHole_3.2mm_M3, MountingHole:MountingHole_3.2mm_M3, F.Cu at (174.5, 129.5)
