File: KiCAD/analog/interface.kicad_sch (KiCad schematic)
At the start: 11 parts, among them J15 Conn_01x03_Pin, J4 8P8C_Shielded, U16 AM26LS32ACN

Commit message: kicad: note incorrect AM26LS32ACN (U16) footprint pinout on interface sheet
Adds a bold text note to interface.kicad_sch documenting which pins of U16
(AM26LS32ACN) are swapped relative to the placed footprint.  No footprint
or netlist changes -- PCB Rev A is already fabricated.  Fix will land in RevB.

Also picks up KiCad's automatic (project "KiCAD" -> "analog") instance-path
rename across all five sub-sheets (cosmetic metadata only).

Co-Authored-By: Claude Sonnet 4.6 <noreply@anthropic.com>
Other:
- note added: "The pinout shown for U16 is incorrect. 1A - 2 1B - 1 1Y - 3 4A - 14 4B - 15 4Y - 13 The remaining pins are correct"
Changed lines of the file:
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@@
+		)
+	)
+	(text "The pinout shown for U16 is incorrect.\n1A - 2\n1B - 1\n1Y - 3\n4A - 14\n4B - 15\n4Y - 13\nThe remaining pins are correct"
+		(exclude_from_sim no)
+		(at 195.072 101.6 0)
+		(effects
+			(font
+				(size 1.27 1.27)
+				(thickness 0.254)
+				(bold yes)
+			)
+			(justify left)
 		)
 	)
@@
 		)
 		(instances
-			(project "KiCAD"
+			(project "analog"
 				(path "/d3de40b8-856b-4fbd-829c-f45ffcd55742/5c3f4a2b-7d1e-4f8b-9c6d-0e8a1b2c3d4e"
 					(reference "#PWR097")
@@
 		)
 		(instances
-			(project "KiCAD"
+			(project "analog"
 				(path "/d3de40b8-856b-4fbd-829c-f45ffcd55742/5c3f4a2b-7d1e-4f8b-9c6d-0e8a1b2c3d4e"
 					(reference "#PWR099")
@@
 		)
 		(instances
-			(project "KiCAD"
+			(project "analog"
 				(path "/d3de40b8-856b-4fbd-829c-f45ffcd55742/5c3f4a2b-7d1e-4f8b-9c6d-0e8a1b2c3d4e"
 					(reference "#PWR092")
@@
 		)
 		(instances
-			(project "KiCAD"
+			(project "analog"
 				(path "/d3de40b8-856b-4fbd-829c-f45ffcd55742/5c3f4a2b-7d1e-4f8b-9c6d-0e8a1b2c3d4e"
 					(reference "#PWR094")
@@
 		)
 		(instances
-			(project "KiCAD"
+			(project "analog"
 				(path "/d3de40b8-856b-4fbd-829c-f45ffcd55742/5c3f4a2b-7d1e-4f8b-9c6d-0e8a1b2c3d4e"
 					(reference "R26")
@@
 		)
 		(instances
-			(project "KiCAD"
+			(project "analog"
 				(path "/d3de40b8-856b-4fbd-829c-f45ffcd55742/5c3f4a2b-7d1e-4f8b-9c6d-0e8a1b2c3d4e"
 					(reference "R27")
@@
 		)
 		(instances
-			(project "KiCAD"
+			(project "analog"
 				(path "/d3de40b8-856b-4fbd-829c-f45ffcd55742/5c3f4a2b-7d1e-4f8b-9c6d-0e8a1b2c3d4e"
 					(reference "#PWR089")
@@
 		)
 		(instances
-			(project "KiCAD"
+			(project "analog"
 				(path "/d3de40b8-856b-4fbd-829c-f45ffcd55742/5c3f4a2b-7d1e-4f8b-9c6d-0e8a1b2c3d4e"
 					(reference "R100")
@@
 		)
 		(instances
-			(project "KiCAD"
+			(project "analog"
 				(path "/d3de40b8-856b-4fbd-829c-f45ffcd55742/5c3f4a2b-7d1e-4f8b-9c6d-0e8a1b2c3d4e"
 					(reference "R101")
@@
 		)
 		(instances
-			(project "KiCAD"
+			(project "analog"
 				(path "/d3de40b8-856b-4fbd-829c-f45ffcd55742/5c3f4a2b-7d1e-4f8b-9c6d-0e8a1b2c3d4e"
 					(reference "#PWR093")
@@
 		)
 		(instances
-			(project "KiCAD"
+			(project "analog"
 				(path "/d3de40b8-856b-4fbd-829c-f45ffcd55742/5c3f4a2b-7d1e-4f8b-9c6d-0e8a1b2c3d4e"
 					(reference "#PWR091")
@@
 		)
 		(instances
-			(project "KiCAD"
+			(project "analog"
 				(path "/d3de40b8-856b-4fbd-829c-f45ffcd55742/5c3f4a2b-7d1e-4f8b-9c6d-0e8a1b2c3d4e"
 					(reference "#PWR095")
@@
 		)
 		(instances
-			(project "KiCAD"
+			(project "analog"
 				(path "/d3de40b8-856b-4fbd-829c-f45ffcd55742/5c3f4a2b-7d1e-4f8b-9c6d-0e8a1b2c3d4e"
 					(reference "R29")
@@
 		)
 		(instances
-			(project "KiCAD"
+			(project "analog"
 				(path "/d3de40b8-856b-4fbd-829c-f45ffcd55742/5c3f4a2b-7d1e-4f8b-9c6d-0e8a1b2c3d4e"
 					(reference "#PWR096")
@@
 		)
 		(instances
-			(project "KiCAD"
+			(project "analog"
 				(path "/d3de40b8-856b-4fbd-829c-f45ffcd55742/5c3f4a2b-7d1e-4f8b-9c6d-0e8a1b2c3d4e"
 					(reference "#PWR090")
@@
 		)
 		(instances
-			(project "KiCAD"
+			(project "analog"
 				(path "/d3de40b8-856b-4fbd-829c-f45ffcd55742/5c3f4a2b-7d1e-4f8b-9c6d-0e8a1b2c3d4e"
 					(reference "#PWR098")
@@
 		)
 		(instances
-			(project "KiCAD"
+			(project "analog"
 				(path "/d3de40b8-856b-4fbd-829c-f45ffcd55742/5c3f4a2b-7d1e-4f8b-9c6d-0e8a1b2c3d4e"
 					(reference "C35")
@@
 		)
 		(instances
-			(project "KiCAD"
+			(project "analog"
 				(path "/d3de40b8-856b-4fbd-829c-f45ffcd55742/5c3f4a2b-7d1e-4f8b-9c6d-0e8a1b2c3d4e"
 					(reference "C34")
@@
 		)
 		(instances
-			(project "KiCAD"
+			(project "analog"
 				(path "/d3de40b8-856b-4fbd-829c-f45ffcd55742/5c3f4a2b-7d1e-4f8b-9c6d-0e8a1b2c3d4e"
 					(reference "R28")
@@
 		)
 		(instances
-			(project "KiCAD"
+			(project "analog"
 				(path "/d3de40b8-856b-4fbd-829c-f45ffcd55742/5c3f4a2b-7d1e-4f8b-9c6d-0e8a1b2c3d4e"
 					(reference "J4")
@@
 		)
 		(instances
-			(project "KiCAD"
+			(project "analog"
 				(path "/d3de40b8-856b-4fbd-829c-f45ffcd55742/5c3f4a2b-7d1e-4f8b-9c6d-0e8a1b2c3d4e"
 					(reference "J15")
@@
 		)
 		(instances
-			(project "KiCAD"
+			(project "analog"
 				(path "/d3de40b8-856b-4fbd-829c-f45ffcd55742/5c3f4a2b-7d1e-4f8b-9c6d-0e8a1b2c3d4e"
 					(reference "#PWR0119")
@@
 		)
 		(instances
-			(project "KiCAD"
+			(project "analog"
 				(path "/d3de40b8-856b-4fbd-829c-f45ffcd55742/5c3f4a2b-7d1e-4f8b-9c6d-0e8a1b2c3d4e"
 					(reference "U16")
