File: KiCAD/analog/buffer_keyer.kicad_sch (KiCad schematic)
At the start: 92 parts, among them J1 Conn_01x02_Pin, J13 Conn_01x05, J16 Conn_01x05, T1 2N3906, T2 2N3906, U15 LM7805_TO220, U19 L79L08_TO92, U20 ICL7660S, U3 MC1496, U4 MCP4921, U6 LM7171xIN, U7 LM7171xIN, U8 MCP4728

Commit message: revB: encoder retry + J1 Phoenix Contact footprint + schematic updates
- firmware rev 20: seesaw ATTINY intermittent NAK fix -- retry read_delta
  up to 3x before skipping poll cycle; counts accumulate in seesaw so
  no detents are lost across retries
- KiCAD/analog/buffer_keyer.kicad_sch: J1 footprint changed from generic
  PinHeader_1x02_P2.54mm to TerminalBlock_Phoenix_MKDS-1,5-2_1x02_P5.00mm_Horizontal
  (Phoenix Contact 1715022, 5mm pitch, 1.3mm drill); datasheet URL added
- KiCAD/analog schematics: capture pending schematic edits from Rev A bring-up
- Documentation: add Phoenix Contact MKDS 1,5/2 datasheet (1715022)

Co-Authored-By: Claude Sonnet 4.6 (1M context) <noreply@anthropic.com>
Parts:
- J1: footprint Connector_PinHeader_2.54mm:PinHeader_1x02_P2.54mm_Vertical -> TerminalBlock_Phoenix:TerminalBlock_Phoenix_MKDS-1,5-2_1x02_P5.00mm_Horizontal

Commit message: KiCad revB: widen TO-92 footprint to Inline_Wide (2.54 mm pitch)
Change Package_TO_SOT_THT:TO-92_Inline to TO-92_Inline_Wide on all
TO-92 parts across the analog board schematics:
  - 2N3904 (untitled.kicad_sch, 2 instances)
  - 2N3906 (buffer_keyer.kicad_sch, 2 instances + L79L08 regulator)
  - J310   (vfo.kicad_sch, 1 instance)
  - 2N7000 (arduino.kicad_sch, 4 instances)
  - L79L08_TO92 (buffer_keyer.kicad_sch, 1 instance)

Inline_Wide has 2.54 mm pad pitch vs 1.27 mm — matches the ~2.6 mm
lead spacing of tape-supplied TO-92 parts and avoids the narrow-lead
hand-soldering difficulty.

Co-Authored-By: Claude Sonnet 4.6 <noreply@anthropic.com>
Parts:
- T1, T2, U19: footprint Package_TO_SOT_THT:TO-92_Inline -> Package_TO_SOT_THT:TO-92_Inline_Wide
Changed lines of the file:
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@@
 			)
 		)
-		(property "Footprint" "Package_TO_SOT_THT:TO-92_Inline"
+		(property "Footprint" "Package_TO_SOT_THT:TO-92_Inline_Wide"
 			(at 201.93 133.35 0)
 			(hide yes)
@@
 			)
 		)
-		(property "Footprint" "Package_TO_SOT_THT:TO-92_Inline"
+		(property "Footprint" "Package_TO_SOT_THT:TO-92_Inline_Wide"
 			(at 54.61 103.505 0)
 			(hide yes)
@@
 			)
 		)
-		(property "Footprint" "Package_TO_SOT_THT:TO-92_Inline"
+		(property "Footprint" "Package_TO_SOT_THT:TO-92_Inline_Wide"
 			(at 109.22 103.505 0)
 			(hide yes)
