File: KiCAD/analog/vfo.kicad_sch (KiCad schematic)
At the start: 20 parts, among them Q1 J310, U1 Si5351A_Breakout

Commit message: revB: encoder retry + J1 Phoenix Contact footprint + schematic updates
- firmware rev 20: seesaw ATTINY intermittent NAK fix -- retry read_delta
  up to 3x before skipping poll cycle; counts accumulate in seesaw so
  no detents are lost across retries
- KiCAD/analog/buffer_keyer.kicad_sch: J1 footprint changed from generic
  PinHeader_1x02_P2.54mm to TerminalBlock_Phoenix_MKDS-1,5-2_1x02_P5.00mm_Horizontal
  (Phoenix Contact 1715022, 5mm pitch, 1.3mm drill); datasheet URL added
- KiCAD/analog schematics: capture pending schematic edits from Rev A bring-up
- Documentation: add Phoenix Contact MKDS 1,5/2 datasheet (1715022)

Co-Authored-By: Claude Sonnet 4.6 (1M context) <noreply@anthropic.com>
Parts:
- L2, L6: value 736nH -> 680nH
- L4: value 736nH -> 790nH
Changed lines of the file:
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@@
 		)
 		(instances
-			(project "KiCAD"
+			(project "analog"
 				(path "/d3de40b8-856b-4fbd-829c-f45ffcd55742/c08cbce4-6e06-48f3-b334-a48b1cc09989"
 					(reference "#PWR02")
@@
 		)
 		(instances
-			(project "KiCAD"
+			(project "analog"
 				(path "/d3de40b8-856b-4fbd-829c-f45ffcd55742/c08cbce4-6e06-48f3-b334-a48b1cc09989"
 					(reference "Q1")
@@
 		)
 		(instances
-			(project "KiCAD"
+			(project "analog"
 				(path "/d3de40b8-856b-4fbd-829c-f45ffcd55742/c08cbce4-6e06-48f3-b334-a48b1cc09989"
 					(reference "#PWR01")
@@
 		)
 		(instances
-			(project "KiCAD"
+			(project "analog"
 				(path "/d3de40b8-856b-4fbd-829c-f45ffcd55742/c08cbce4-6e06-48f3-b334-a48b1cc09989"
 					(reference "#PWR06")
@@
 		)
 		(instances
-			(project "KiCAD"
+			(project "analog"
 				(path "/d3de40b8-856b-4fbd-829c-f45ffcd55742/c08cbce4-6e06-48f3-b334-a48b1cc09989"
 					(reference "CF7")
@@
 		)
 		(instances
-			(project "KiCAD"
+			(project "analog"
 				(path "/d3de40b8-856b-4fbd-829c-f45ffcd55742/c08cbce4-6e06-48f3-b334-a48b1cc09989"
 					(reference "CF3")
@@
 			)
 		)
-		(property "Value" "736nH"
+		(property "Value" "680nH"
 			(at 163.83 58.42 90)
 			(show_name no)
@@
 		)
 		(instances
-			(project "KiCAD"
+			(project "analog"
 				(path "/d3de40b8-856b-4fbd-829c-f45ffcd55742/c08cbce4-6e06-48f3-b334-a48b1cc09989"
 					(reference "L6")
@@
 		)
 		(instances
-			(project "KiCAD"
+			(project "analog"
 				(path "/d3de40b8-856b-4fbd-829c-f45ffcd55742/c08cbce4-6e06-48f3-b334-a48b1cc09989"
 					(reference "RP3")
@@
 		)
 		(instances
-			(project "KiCAD"
+			(project "analog"
 				(path "/d3de40b8-856b-4fbd-829c-f45ffcd55742/c08cbce4-6e06-48f3-b334-a48b1cc09989"
 					(reference "RS1")
@@
 		)
 		(instances
-			(project "KiCAD"
+			(project "analog"
 				(path "/d3de40b8-856b-4fbd-829c-f45ffcd55742/c08cbce4-6e06-48f3-b334-a48b1cc09989"
 					(reference "#PWR07")
@@
 		)
 		(instances
-			(project "KiCAD"
+			(project "analog"
 				(path "/d3de40b8-856b-4fbd-829c-f45ffcd55742/c08cbce4-6e06-48f3-b334-a48b1cc09989"
 					(reference "#PWR03")
@@
 		)
 		(instances
-			(project "KiCAD"
+			(project "analog"
 				(path "/d3de40b8-856b-4fbd-829c-f45ffcd55742/c08cbce4-6e06-48f3-b334-a48b1cc09989"
 					(reference "R17")
@@
 		)
 		(instances
-			(project "KiCAD"
+			(project "analog"
 				(path "/d3de40b8-856b-4fbd-829c-f45ffcd55742/c08cbce4-6e06-48f3-b334-a48b1cc09989"
 					(reference "RT1")
@@
 		)
 		(instances
-			(project "KiCAD"
+			(project "analog"
 				(path "/d3de40b8-856b-4fbd-829c-f45ffcd55742/c08cbce4-6e06-48f3-b334-a48b1cc09989"
 					(reference "C44")
@@
 		)
 		(instances
-			(project "KiCAD"
+			(project "analog"
 				(path "/d3de40b8-856b-4fbd-829c-f45ffcd55742/c08cbce4-6e06-48f3-b334-a48b1cc09989"
 					(reference "RD1")
@@
 		)
 		(instances
-			(project "KiCAD"
+			(project "analog"
 				(path "/d3de40b8-856b-4fbd-829c-f45ffcd55742/c08cbce4-6e06-48f3-b334-a48b1cc09989"
 					(reference "TP1")
@@
 		)
 		(instances
-			(project "KiCAD"
+			(project "analog"
 				(path "/d3de40b8-856b-4fbd-829c-f45ffcd55742/c08cbce4-6e06-48f3-b334-a48b1cc09989"
 					(reference "#PWR08")
@@
 			)
 		)
-		(property "Value" "736nH"
+		(property "Value" "790nH"
 			(at 142.24 58.42 90)
 			(show_name no)
@@
 		)
 		(instances
-			(project "KiCAD"
+			(project "analog"
 				(path "/d3de40b8-856b-4fbd-829c-f45ffcd55742/c08cbce4-6e06-48f3-b334-a48b1cc09989"
 					(reference "L4")
@@
 		)
 		(instances
-			(project "KiCAD"
+			(project "analog"
 				(path "/d3de40b8-856b-4fbd-829c-f45ffcd55742/c08cbce4-6e06-48f3-b334-a48b1cc09989"
 					(reference "C_IN1")
@@
 		)
 		(instances
-			(project "KiCAD"
+			(project "analog"
 				(path "/d3de40b8-856b-4fbd-829c-f45ffcd55742/c08cbce4-6e06-48f3-b334-a48b1cc09989"
 					(reference "CF1")
@@
 		)
 		(instances
-			(project "KiCAD"
+			(project "analog"
 				(path "/d3de40b8-856b-4fbd-829c-f45ffcd55742/c08cbce4-6e06-48f3-b334-a48b1cc09989"
 					(reference "#PWR04")
@@
 		)
 		(instances
-			(project "KiCAD"
+			(project "analog"
 				(path "/d3de40b8-856b-4fbd-829c-f45ffcd55742/c08cbce4-6e06-48f3-b334-a48b1cc09989"
 					(reference "#PWR074")
@@
 		)
 		(instances
-			(project "KiCAD"
+			(project "analog"
 				(path "/d3de40b8-856b-4fbd-829c-f45ffcd55742/c08cbce4-6e06-48f3-b334-a48b1cc09989"
 					(reference "U1")
@@
 		)
 		(instances
-			(project "KiCAD"
+			(project "analog"
 				(path "/d3de40b8-856b-4fbd-829c-f45ffcd55742/c08cbce4-6e06-48f3-b334-a48b1cc09989"
 					(reference "#PWR05")
@@
 		)
 		(instances
-			(project "KiCAD"
+			(project "analog"
 				(path "/d3de40b8-856b-4fbd-829c-f45ffcd55742/c08cbce4-6e06-48f3-b334-a48b1cc09989"
 					(reference "#PWR055")
@@
 		)
 		(instances
-			(project "KiCAD"
+			(project "analog"
 				(path "/d3de40b8-856b-4fbd-829c-f45ffcd55742/c08cbce4-6e06-48f3-b334-a48b1cc09989"
 					(reference "CC1")
@@
 			)
 		)
-		(property "Value" "736nH"
+		(property "Value" "680nH"
 			(at 120.65 58.42 90)
 			(show_name no)
@@
 		)
 		(instances
-			(project "KiCAD"
+			(project "analog"
 				(path "/d3de40b8-856b-4fbd-829c-f45ffcd55742/c08cbce4-6e06-48f3-b334-a48b1cc09989"
 					(reference "L2")
@@
 		)
 		(instances
-			(project "KiCAD"
+			(project "analog"
 				(path "/d3de40b8-856b-4fbd-829c-f45ffcd55742/c08cbce4-6e06-48f3-b334-a48b1cc09989"
 					(reference "RP1")
@@
 		)
 		(instances
-			(project "KiCAD"
+			(project "analog"
 				(path "/d3de40b8-856b-4fbd-829c-f45ffcd55742/c08cbce4-6e06-48f3-b334-a48b1cc09989"
 					(reference "CF5")
@@
 		)
 		(instances
-			(project "KiCAD"
+			(project "analog"
 				(path "/d3de40b8-856b-4fbd-829c-f45ffcd55742/c08cbce4-6e06-48f3-b334-a48b1cc09989"
 					(reference "RP2")
@@
 		)
 		(instances
-			(project "KiCAD"
+			(project "analog"
 				(path "/d3de40b8-856b-4fbd-829c-f45ffcd55742/c08cbce4-6e06-48f3-b334-a48b1cc09989"
 					(reference "#PWR023")
@@
 		)
 		(instances
-			(project "KiCAD"
+			(project "analog"
 				(path "/d3de40b8-856b-4fbd-829c-f45ffcd55742/c08cbce4-6e06-48f3-b334-a48b1cc09989"
 					(reference "#PWR09")

Commit message: KiCAD/analog/vfo: KiCad embeds Device:C_Polarized symbol cache
KiCad auto-embedded the Device:C_Polarized symbol definition into
vfo.kicad_sch when the schematic was opened.

Co-Authored-By: Claude Sonnet 4.6 (1M context) <noreply@anthropic.com>
Parts:
- added C22: 10uF, symbol Device:C_Polarized
- added C23: 100nF, symbol Device:C
Connections:
- net 3V3: now also C22.1, C23.2
- net GND: now also C22.2, C23.1

Commit message: KiCAD/analog/vfo: assign footprints to C22, C23
C22=10uF  -> CP_Radial_D5.0mm_P2.00mm  (matches all other 10uF on board)
C23=100nF -> C_Disc_D5.0mm_W2.5mm_P5.00mm  (matches all other 100nF on board)

Co-Authored-By: Claude Sonnet 4.6 (1M context) <noreply@anthropic.com>
Parts:
- C22: footprint (none) -> Capacitor_THT:CP_Radial_D5.0mm_P2.00mm
- C23: footprint (none) -> Capacitor_THT:C_Disc_D5.0mm_W2.5mm_P5.00mm
Changed lines of the file:
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@@
 			)
 		)
-		(property "Footprint" ""
+		(property "Footprint" "Capacitor_THT:C_Disc_D5.0mm_W2.5mm_P5.00mm"
 			(at 26.3652 55.88 0)
 			(hide yes)
@@
 			)
 		)
-		(property "Footprint" ""
+		(property "Footprint" "Capacitor_THT:CP_Radial_D5.0mm_P2.00mm"
 			(at 26.3652 63.5 0)
 			(hide yes)

Commit message: schematic: revB encoder interrupt rerouted through CAT6 umbilical
- interface.kicad_sch: ENC_INT global label (input) replaces the old
  direct wire+GND stub; encoder interrupt now travels over the RJ45
  cable with the shield as signal return
- frontpanel.kicad_sch: 4-pin header J (Conn_01x04) added for up to
  3 encoder connections + one test-point pin; ENC_INT_IN label wired in
- arduino.kicad_sch: removed orphaned Conn_Coaxial symbol cache
- vfo.kicad_sch: minor layout/annotation updates

Co-Authored-By: Claude Sonnet 4.6 (1M context) <noreply@anthropic.com>
Parts:
- added TP8: FILTERED_RF, symbol Connector:TestPoint
Connections:
- net at CC1.2, Q1.2 (G), R17.1: now also TP8.1
Changed lines of the file:
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@@
+	)
+	(symbol
+		(lib_id "Connector:TestPoint")
+		(at 195.58 62.23 0)
+		(unit 1)
+		(body_style 1)
+		(exclude_from_sim no)
+		(in_bom yes)
+		(on_board yes)
+		(in_pos_files yes)
+		(dnp no)
+		(property "Reference" "TP8"
+			(at 192.024 54.61 0)
+			(show_name no)
+			(do_not_autoplace no)
+			(effects
+				(font
+					(size 1.27 1.27)
+				)
+				(justify left)
+			)
+		)
+		(property "Value" "FILTERED_RF"
+			(at 192.024 57.15 0)
+			(show_name no)
+			(do_not_autoplace no)
+			(effects
+				(font
+					(size 1.27 1.27)
+				)
+				(justify left)
+			)
+		)
+		(property "Footprint" ""
+			(at 200.66 62.23 0)
+			(hide yes)
+			(show_name no)
+			(do_not_autoplace no)
+			(effects
+				(font
+					(size 1.27 1.27)
+				)
+			)
+		)
+		(property "Datasheet" ""
+			(at 200.66 62.23 0)
+			(hide yes)
+			(show_name no)
+			(do_not_autoplace no)
+			(effects
+				(font
+					(size 1.27 1.27)
+				)
+			)
+		)
+		(property "Description" "test point"
+			(at 195.58 62.23 0)
+			(hide yes)
+			(show_name no)
+			(do_not_autoplace no)
+			(effects
+				(font
+					(size 1.27 1.27)
+				)
+			)
+		)
+		(pin "1"
+		)
+		(instances
+			(project "analog"
+				(path "/d3de40b8-856b-4fbd-829c-f45ffcd55742/c08cbce4-6e06-48f3-b334-a48b1cc09989"
+					(reference "TP8")
+					(unit 1)
+				)
+			)
+		)
 	)
 	(symbol

Commit message: KiCad revB: widen TO-92 footprint to Inline_Wide (2.54 mm pitch)
Change Package_TO_SOT_THT:TO-92_Inline to TO-92_Inline_Wide on all
TO-92 parts across the analog board schematics:
  - 2N3904 (untitled.kicad_sch, 2 instances)
  - 2N3906 (buffer_keyer.kicad_sch, 2 instances + L79L08 regulator)
  - J310   (vfo.kicad_sch, 1 instance)
  - 2N7000 (arduino.kicad_sch, 4 instances)
  - L79L08_TO92 (buffer_keyer.kicad_sch, 1 instance)

Inline_Wide has 2.54 mm pad pitch vs 1.27 mm — matches the ~2.6 mm
lead spacing of tape-supplied TO-92 parts and avoids the narrow-lead
hand-soldering difficulty.

Co-Authored-By: Claude Sonnet 4.6 <noreply@anthropic.com>
Parts:
- Q1: footprint Package_TO_SOT_THT:TO-92_Inline -> Package_TO_SOT_THT:TO-92_Inline_Wide
Changed lines of the file:
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@@
 			)
 		)
-		(property "Footprint" "Package_TO_SOT_THT:TO-92_Inline"
+		(property "Footprint" "Package_TO_SOT_THT:TO-92_Inline_Wide"
 			(at 201.93 62.23 0)
 			(hide yes)
