File: KiCAD/analog/lpf.kicad_sch (KiCad schematic)
At the start: 0 parts

Commit message: KiCad revC: 4-band LPF bank populated + pad values + A_L units fix
Analog board revC: the LPF sheet is now fully populated with the
4-band relay-switched LPF bank architecture discussed in prior
sessions.  VFO sheet refactored to remove the old single-LPF stage.

LPF bank (lpf.kicad_sch):
  - 4 branches tied to a common input bus from U2 (LM7171 buffer).
    Common bus driven through C9 100nF; U2 non-inverting gain = 5.7.
  - Per-branch: 10 dB pi attenuator (100/68/100 ohm) -> 7-element
    Chebyshev CLCLCLC LPF (0.1 dB ripple, 50 ohm) -> 50 ohm RT
    terminator -> SPST relay (K1-K4) -> common output bus
    "Conditioned RF" -> R39 (0R) -> U10 input on VFO sheet.
  - Relay drive: 2N7000 low-side switcher (Q1/Q3/Q8/Q9) + 1N4148
    flyback diode (D7-D10) + screw terminal (J16/J25/J26/J27) per
    relay for coil wire termination.
  - LPF components: CF3-CF21 and L4-L17 populated with 20 m values
    (220 pF / 390 pF / 680 nH / 790 nH) on all four branches.
    Other-band values TBD per Documentation/lpf_component_values.md.
  - Pi pad resistors are now 100/68/100 (10 dB) rather than the
    initially-populated 62/240/62 (20 dB).  Reasoning: with permanent
    50 ohm termination at each LPF output and relay-based output
    switching, the pi pads are only providing impedance isolation at
    the common input bus, not inter-LPF signal isolation (which is
    handled by relay off-isolation of ~40 dB per open contact).
    10 dB is sufficient and recovers ~10 dB of noise margin.

VFO sheet (vfo_complete.kicad_sch):
  - Old inline LPF removed; VFO now feeds C10 -> U2 (on LPF sheet)
    via sheet-boundary net.
  - U10/U11/U12 LM7171 chain (post-LPF-bank amplifier + PP driver
    pair) retained.

Documentation/lpf_component_values.md (new):
  - Component values for all four bands (20/17/15/10 m).
  - 7-element Chebyshev CLCLCLC, 0.1 dB ripple, 50 ohm.
  - Per-band tables for T50-6 and T68-6 turn counts.
  - Notes on A_L unit convention (catalogs use uH/100T^2 not nH/N^2).

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
Parts:
- added C10: 10nF, symbol Device:C
- added C9: 100nF, symbol Device:C
- added C91, C96: 10uF, Capacitor_THT:CP_Radial_D5.0mm_P2.00mm, symbol Device:C_Polarized_US
- added C93, C97: 100nF, Capacitor_THT:C_Disc_D5.0mm_W2.5mm_P5.00mm, symbol Device:C_US
- added C94, C98: 10nF, Capacitor_THT:C_Disc_D6.0mm_W2.5mm_P5.00mm, symbol Device:C_US
- added C95: 2pF, xmitter:C_Axial_Kemet_Aximax_C41X_L4.5mm_D2.6mm_P7.62mm_Horizontal, symbol Device:C_US
- added CF10, CF13, CF14, CF17, CF18, CF21, CF3, CF9: 220pF, Capacitor_THT:C_Disc_D6.0mm_W2.5mm_P5.00mm, symbol Device:C
- added CF11, CF12, CF15, CF16, CF19, CF20, CF5, CF7: 390pF, Capacitor_THT:C_Disc_D7.5mm_W2.5mm_P5.00mm, symbol Device:C
- added D10, D7, D8, D9: 1N4148, Diode_THT:D_DO-35_SOD27_P7.62mm_Horizontal, symbol Diode:1N4148
- added J16, J25, J26, J27: Screw_Terminal_01x02, symbol Connector:Screw_Terminal_01x02
- added J28: Filter In, Connector_Coaxial:SMA_Amphenol_132134_Vertical, symbol Connector:Conn_Coaxial_Small
- added K1, K2, K3, K4: Relay_RSS-SR042P, xmitter:Relay_SPST_RelComm_RSS-SR042P, symbol xmitter:Relay_SPST_RSS-SR042P
- added L10, L13, L16, L6: 790nH, xmitter:T68-6_Vertical_HandWound, symbol Device:L_Ferrite
- added L11, L12, L14, L15, L17, L4, L7, L9: 680nH, xmitter:T68-6_Flat_HandWound, symbol Device:L_Ferrite
- added Q1, Q3, Q8, Q9: 2N7000, Package_TO_SOT_THT:TO-92_Inline, symbol Transistor_FET:2N7000
- added R11: 1K, symbol Device:R_US
- added R42: 1K, Resistor_THT:R_Axial_DIN0207_L6.3mm_D2.5mm_P10.16mm_Horizontal, symbol Device:R_US
- added R43: 4.7K, Resistor_THT:R_Axial_DIN0207_L6.3mm_D2.5mm_P10.16mm_Horizontal, symbol Device:R_US
- added RP10, RP12, RP13, RP15, RP16, RP18, RP7, RP9: 100R, Resistor_THT:R_Axial_DIN0207_L6.3mm_D2.5mm_P10.16mm_Horizontal, symbol Device:R_US
- added RP11, RP14, RP17, RP8: 68R, Resistor_THT:R_Axial_DIN0207_L6.3mm_D2.5mm_P10.16mm_Horizontal, symbol Device:R_US
- added RT3, RT4, RT5, RT6: 50R, Resistor_THT:R_Axial_DIN0207_L6.3mm_D2.5mm_P10.16mm_Horizontal, symbol Device:R_US
- added U2: LM7171xIN, Package_DIP:DIP-8_W7.62mm, symbol Amplifier_Operational:LM7171xIN
Connections:
- new net: C95.1, R42.1, R43.1, U2.2 (-)
- new net: C10.2, R11.1, U2.3 (+)
- new net: C9.1, C95.2, R43.2, U2.6
- new net: CF12.1, L10.2, L11.1
- new net: CF13.1, K3.1 (RF_A), L11.2, RT4.1
- new net: CF9.1, K4.1 (RF_A), L9.2, RT3.1
- new net: D8.2 (A), J25.2 (Pin_2), Q3.3 (D)
- new net: C9.2, J28.1 (In), RP10.1, RP11.1, RP13.1, RP14.1, RP16.1, RP17.1, RP7.1, RP8.1
- new net: CF18.1, L15.1, RP17.2, RP18.1
- new net: CF19.1, L15.2, L16.1
- new net: D7.2 (A), J16.2 (Pin_2), Q1.3 (D)
- new net: CF5.1, L4.2, L6.1
- new net: CF11.1, L10.1, L7.2
- new net: D9.2 (A), J26.2 (Pin_2), Q8.3 (D)
- new net: CF10.1, L7.1, RP11.2, RP12.1
- new net: CF3.1, L4.1, RP8.2, RP9.1
- new net: CF14.1, L12.1, RP14.2, RP15.1
- new net: CF20.1, L16.2, L17.1
- new net: D10.2 (A), J27.2 (Pin_2), Q9.3 (D)
- new net: CF21.1, K1.1 (RF_A), L17.2, RT6.1
- new net: CF16.1, L13.2, L14.1
- new net: CF17.1, K2.1 (RF_A), L14.2, RT5.1
- new net: CF15.1, L12.2, L13.1
- new net: CF7.1, L6.2, L9.1
- new net +12V: C96.1, C97.1, C98.1, U2.7 (V+)
- new net +28V: D10.1 (K), D7.1 (K), D8.1 (K), D9.1 (K), J16.1 (Pin_1), J25.1 (Pin_1), J26.1 (Pin_1), J27.1 (Pin_1)
- new net -12V: C91.1, C93.1, C94.1, U2.4 (V-)
- new net Conditioned RF: K1.2 (RF_B), K2.2 (RF_B), K3.2 (RF_B), K4.2 (RF_B)
- new net GND: C91.2, C93.2, C94.2, C96.2, C97.2, C98.2, CF10.2, CF11.2, CF12.2, CF13.2, CF14.2, CF15.2, CF16.2, CF17.2, CF18.2, CF19.2, CF20.2, CF21.2, CF3.2, CF5.2, CF7.2, CF9.2, J28.2 (Ext), K1.3 (SHIELD), K2.3 (SHIELD), K3.3 (SHIELD), K4.3 (SHIELD), Q1.1 (S), Q3.1 (S), Q8.1 (S), Q9.1 (S), R11.2, R42.2, RP10.2, RP12.2, RP13.2, RP15.2, RP16.2, RP18.2, RP7.2, RP9.2, RT3.2, RT4.2, RT5.2, RT6.2
- new net RLY_10: Q9.2 (G)
- new net RLY_15: Q3.2 (G)
- new net RLY_17: Q8.2 (G)
- new net RLY_20: Q1.2 (G)
- new net Raw RF: C10.1

Commit message: KiCad revC: toroid footprints with zip-tie holes + T50-6 variants
Four hand-wound toroid footprints -- flat and vertical variants for
both T68-6 and T50-6 cores -- each with NPTH holes sized for 0.122 in
zip ties to secure the toroid to the PCB after winding.

Vertical variants (both T50-6 and T68-6):
  - Two 3.1 mm NPTH tie holes at (0, +-3.5) on the midline through
    the toroid's rotation axis.  A single zip tie wraps over the top
    of the standing disc in the Y direction (crossing the thin H
    dimension, not the wide OD).
  - Wire pads at (+-3.0, +-4.5) -- moved laterally and inward from
    an earlier (+-2.0, +-6.0) layout to allow tighter Y-direction
    packing of multiple toroids in a bank.  Clearance pad <-> tie
    hole = 0.76 mm.
  - Courtyard tight at +-5.6 mm Y, OD-limited in X.

Flat variants (both T68-6 and T50-6):
  - Four 3.1 mm NPTH tie holes in two pairs: each tie has one hole
    just inside the ID and one hole just outside the OD, with the
    tie wrapping across the donut wall on one side.  Two ties on
    opposite +-X sides clamp the toroid without crossing the ID
    center.  Tie direction = X axis (90 deg from the Y-axis
    wire-pad direction).
  - T50-6 Flat: ties at (+-2.0, 0) and (+-7.5, 0).
  - T68-6 Flat: ties at (+-2.9, 0) and (+-9.9, 0).
  - Courtyards expanded to include the full toroid OD + 24 AWG wire
    bulge on all sides.  Specifically fixed a serious bug where the
    T68-6 Flat courtyard was clipping the toroid at Y+6.6 (toroid
    OD is at Y+8.77).  Now Y+ extends to +9.9 (T68) and +7.5 (T50),
    both with 0.5 mm margin beyond the wire bulge.

T68-6 footprint descriptions updated to show the A_L unit convention
(4.7 nH/N^2 = 47 microH per 100 turns^2) -- see memory lesson
lesson_toroid_AL_units for the factor-of-10 trap this avoids.

Also touched: KiCad project file (pin table or similar auto-updates)
and lpf.kicad_sch (user's in-progress schematic edits).

Co-Authored-By: Claude Opus 4.7 <noreply@anthropic.com>
Parts:
- L4, L9: footprint xmitter:T68-6_Flat_HandWound -> xmitter:T50-6_Vertical_HandWound
- L6: footprint xmitter:T68-6_Vertical_HandWound -> xmitter:T50-6_Flat_HandWound
Changed lines of the file:
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@@
 			)
 		)
-		(property "Footprint" "xmitter:T68-6_Vertical_HandWound"
+		(property "Footprint" "xmitter:T50-6_Flat_HandWound"
 			(at 134.62 38.1 0)
 			(hide yes)
@@
 			)
 		)
-		(property "Footprint" "xmitter:T68-6_Flat_HandWound"
+		(property "Footprint" "xmitter:T50-6_Vertical_HandWound"
 			(at 113.03 38.1 0)
 			(hide yes)
@@
 			)
 		)
-		(property "Footprint" "xmitter:T68-6_Flat_HandWound"
+		(property "Footprint" "xmitter:T50-6_Vertical_HandWound"
 			(at 156.21 38.1 0)
 			(hide yes)
