File: KiCAD/analog/analog.kicad_pcb (KiCad board)
At the start: 2 copper layers, 130 x 170 mm, 151 parts, among them J1 Conn_01x02_Pin, J13 Conn_01x05, J15 Conn_01x03_Pin, J16 Conn_01x05, J4 8P8C_Shielded, J5 ENC_INT if needed, J6 TX/RX, J7 HV, J8 HV_INRUSH_BYPASS, J9 TR_SENSE, Q1 J310, Q4 2N7000, Q5 2N7000, Q6 2N7000, Q7 2N7000, T1 2N3906, T2 2N3906, U1 Si5351A_Breakout, U15 LM7805_TO220, U16 AM26LS32ACN, U17 Adafruit_PCF8575_Breakout, U18 CD14538B, U19 L79L08_TO92, U20 ICL7660S, U3 MC1496, U4 MCP4921, U6 LM7171xIN, U7 LM7171xIN, U8 MCP4728

Commit message: KiCad revB: remove obsolete VFO sheets, add J3 footprint, add datasheets
- analog.kicad_sch: dropped VFO and VFO_Buffer_keyer sheets (legacy
  stubs superseded by VFO_Complete). Underlying vfo.kicad_sch and
  buffer_keyer.kicad_sch files deleted. PCB and .kicad_pro refreshed
  to match after Update PCB from Schematic.
- vfo_complete.kicad_sch: J3 (AC input to the +/-12V bridge) gets
  Phoenix Contact MKDS 1,5/2 footprint and a link to the local
  datasheet copy.
- Documentation/Components/: local datasheet copies for parts in the
  current supply bring-up (LM317L, LT1054, LM7800 series, 1N5817,
  2N3904/6, Kemet MLCC leaded, Phoenix Contact 142RHS).
- Documentation/Capacitors_Ordered.xlsx: capacitor inventory summary
  compiled from the Mouser and Digi-Key invoices, for stock-consistent
  reordering.

Co-Authored-By: Claude Opus 4.7 <noreply@anthropic.com>
Parts:
- removed C1: 330pF, Capacitor_THT:C_Disc_D6.0mm_W2.5mm_P5.00mm
- removed C10, C12, C16, C2, C20, C21, C39, C40, C44, C45, C46, C5, C51, C54, C55, C6, C8, C_IN2, C_IN3, C_OP_OUT1, C_OP_OUT2, Cx1: 100nF, Capacitor_THT:C_Disc_D5.0mm_W2.5mm_P5.00mm
- removed C11, C19, C4, C48, C50, C7, C9: 10uF, Capacitor_THT:CP_Radial_D5.0mm_P2.00mm
- removed C13, C14, C15: 1uF, Capacitor_THT:C_Rect_L7.2mm_W4.5mm_P5.00mm
- removed C17, C18: 0.33uF, xmitter:Kyocera_SR20_MLCC
- removed C3: 680nF, Capacitor_THT:C_Rect_L13.0mm_W6.0mm_P10.00mm_FKS3_FKP3_MKS4
- removed C47, C53: 0.1uF, Capacitor_THT:C_Disc_D5.0mm_W2.5mm_P5.00mm
- removed C49: 100uF, Capacitor_THT:CP_Radial_D6.3mm_P2.50mm
- removed C52: 0.33uF, Capacitor_THT:C_Rect_L7.0mm_W3.5mm_P5.00mm
- removed CC1, C_IN1: 10nF, Capacitor_THT:C_Disc_D5.0mm_W2.5mm_P5.00mm
- removed CF1, CF7: 220pF, Capacitor_THT:C_Disc_D6.0mm_W2.5mm_P5.00mm
- removed CF3, CF5: 390pF, Capacitor_THT:C_Disc_D7.5mm_W2.5mm_P5.00mm
- removed J1: Conn_01x02_Pin, Connector_PinHeader_2.54mm:PinHeader_1x02_P2.54mm_Vertical
- removed J13, J16: Conn_01x05, Connector_PinHeader_2.54mm:PinHeader_1x05_P2.54mm_Vertical
- removed L2, L6: 736nH, xmitter:T68-6_Flat_HandWound
- removed L4: 736nH, xmitter:T68-6_Vertical_HandWound
- removed L7: 22uH, Inductor_THT:L_Axial_L7.0mm_D3.3mm_P10.16mm_Horizontal_Fastron_MICC
- removed Q1: J310, Package_TO_SOT_THT:TO-92_Inline
- removed R1, R3, R4: 51R, Resistor_THT:R_Axial_DIN0207_L6.3mm_D2.5mm_P10.16mm_Horizontal
- removed R10, R5, R7, R9: 8K2, Resistor_THT:R_Axial_DIN0207_L6.3mm_D2.5mm_P10.16mm_Horizontal
- removed R11, R12: 22K, Resistor_THT:R_Axial_DIN0207_L6.3mm_D2.5mm_P10.16mm_Horizontal
- removed R13: 1K5, Resistor_THT:R_Axial_DIN0207_L6.3mm_D2.5mm_P10.16mm_Horizontal
- removed R14, R15: 100K, Resistor_THT:R_Axial_DIN0207_L6.3mm_D2.5mm_P10.16mm_Horizontal
- removed R16: 10R, Resistor_THT:R_Axial_DIN0207_L6.3mm_D2.5mm_P10.16mm_Horizontal
- removed R17, RG_OP1, RG_OP2: 10K, Resistor_THT:R_Axial_DIN0207_L6.3mm_D2.5mm_P10.16mm_Horizontal
- removed R2: 6K8, Resistor_THT:R_Axial_DIN0207_L6.3mm_D2.5mm_P10.16mm_Horizontal
- removed R6, R8: 2K7, Resistor_THT:R_Axial_DIN0207_L6.3mm_D2.5mm_P10.16mm_Horizontal
- removed RD1: 270R, Resistor_THT:R_Axial_DIN0207_L6.3mm_D2.5mm_P10.16mm_Horizontal
- removed REF** (x4): MountingHole_3.2mm_M3, MountingHole:MountingHole_3.2mm_M3
- removed RF_OP1, RF_OP2: 30K, Resistor_THT:R_Axial_DIN0207_L6.3mm_D2.5mm_P10.16mm_Horizontal
- removed RLA1, RLB1: 3K9, Resistor_THT:R_Axial_DIN0207_L6.3mm_D2.5mm_P10.16mm_Horizontal
- removed RP1, RP3: 62R, Resistor_THT:R_Axial_DIN0207_L6.3mm_D2.5mm_P10.16mm_Horizontal
- removed RP2: 240R, Resistor_THT:R_Axial_DIN0207_L6.3mm_D2.5mm_P10.16mm_Horizontal
- removed RS1: 0R, Resistor_THT:R_Axial_DIN0207_L6.3mm_D2.5mm_P10.16mm_Horizontal
- removed RT1: 50R, Resistor_THT:R_Axial_DIN0207_L6.3mm_D2.5mm_P10.16mm_Horizontal
- removed R_INJ1, R_INJ2: 330K, Resistor_THT:R_Axial_DIN0207_L6.3mm_D2.5mm_P10.16mm_Horizontal
- removed Re1: 2K, Resistor_THT:R_Axial_DIN0207_L6.3mm_D2.5mm_P10.16mm_Horizontal
- removed T1, T2: 2N3906, Package_TO_SOT_THT:TO-92_Inline
- removed TP1: RAW_RF, Connector_PinHeader_2.54mm:PinHeader_1x01_P2.54mm_Vertical
- removed TP12: LDAC, Connector_PinHeader_2.54mm:PinHeader_1x01_P2.54mm_Vertical
- removed TP13: T2 out, Connector_PinHeader_2.54mm:PinHeader_1x01_P2.54mm_Vertical
- removed TP14: T1 out, Connector_PinHeader_2.54mm:PinHeader_1x01_P2.54mm_Vertical
- removed TP15: Key_Out, Connector_PinHeader_2.54mm:PinHeader_1x01_P2.54mm_Vertical
- removed TP2: MOD_RF+, Connector_PinHeader_2.54mm:PinHeader_1x01_P2.54mm_Vertical
- removed TP20: VEE, Connector_PinHeader_2.54mm:PinHeader_1x01_P2.54mm_Vertical
- removed TP21: +5V, Connector_PinHeader_2.54mm:PinHeader_1x01_P2.54mm_Vertical
- removed TP22: OUT-, Connector_PinHeader_2.54mm:PinHeader_1x01_P2.54mm_Vertical
- removed TP23: OUT+, Connector_PinHeader_2.54mm:PinHeader_1x01_P2.54mm_Vertical
- removed TP3: SCL, Connector_PinHeader_2.54mm:PinHeader_1x01_P2.54mm_Vertical
- removed TP4: SDA, Connector_PinHeader_2.54mm:PinHeader_1x01_P2.54mm_Vertical
- removed TP5: KEY_SIG, Connector_PinHeader_2.54mm:PinHeader_1x01_P2.54mm_Vertical
- removed TP6: CARRIER_IN, Connector_PinHeader_2.54mm:PinHeader_1x01_P2.54mm_Vertical
- removed TP7: MOD_RF-, Connector_PinHeader_2.54mm:PinHeader_1x01_P2.54mm_Vertical
- removed U1: Si5351A_Breakout, xmitter:Adafruit_Si5351A_STEMMA
- removed U15: LM7805_TO220, Package_TO_SOT_THT:TO-220-3_Vertical
- removed U19: L79L08_TO92, Package_TO_SOT_THT:TO-92_Inline
- removed U20: ICL7660S, Package_DIP:DIP-8_W7.62mm
- removed U3: MC1496, Package_DIP:DIP-14_W7.62mm
- removed U4: MCP4921, Package_DIP:DIP-8_W7.62mm
- removed U6, U7: LM7171xIN, Package_DIP:DIP-8_W7.62mm
- removed U8: MCP4728, xmitter:Adafruit_MCP4728_Breakout
- added C24: 100nF, Capacitor_THT:C_Disc_D5.0mm_W2.5mm_P5.00mm, F.Cu at (-86.0, 102.5)
- added C25: 10uF, Capacitor_THT:CP_Radial_D5.0mm_P2.00mm, F.Cu at (-22.3, 103.7)
- added C27: 10uF, Capacitor_THT:C_Rect_L7.2mm_W4.5mm_P5.00mm, F.Cu at (-22.8, 116.5)
- added C28: 1uF, Capacitor_THT:C_Rect_L7.2mm_W4.5mm_P5.00mm, F.Cu at (-22.8, 122.6)
- added C29: 680nF, Capacitor_THT:C_Rect_L13.0mm_W6.0mm_P10.00mm_FKS3_FKP3_MKS4, F.Cu at (-39.1, 81.5)
- added C85: 0.33uF, Capacitor_THT:C_Rect_L7.0mm_W3.5mm_P5.00mm, F.Cu at (-64.3, 134.9)
- added C86: 0.1uF, Capacitor_THT:C_Disc_D5.0mm_W2.5mm_P5.00mm, F.Cu at (-86.0, 106.5)
- added C87: 10uF, Capacitor_THT:CP_Radial_D5.0mm_P2.00mm, F.Cu at (-22.3, 110.2)
- added CC2: 10nF, Capacitor_THT:C_Disc_D5.0mm_W2.5mm_P5.00mm, F.Cu at (-86.0, 110.5)
- added CF2: 220pF, Capacitor_THT:C_Disc_D6.0mm_W2.5mm_P5.00mm, F.Cu at (-86.0, 114.6)
- added CF4: 390pF, Capacitor_THT:C_Disc_D7.5mm_W2.5mm_P5.00mm, F.Cu at (-24.9, 79.7)
- added CF6: 390pF, Capacitor_THT:C_Disc_D7.5mm_W2.5mm_P5.00mm, F.Cu at (-24.9, 83.8)
- added CF8: 220pF, Capacitor_THT:C_Disc_D6.0mm_W2.5mm_P5.00mm, F.Cu at (-86.0, 118.7)
- added C_IN4: 10nF, Capacitor_THT:C_Disc_D5.0mm_W2.5mm_P5.00mm, F.Cu at (-86.0, 122.7)
- added Cx2: 100nF, Capacitor_THT:C_Disc_D5.0mm_W2.5mm_P5.00mm, F.Cu at (-86.0, 126.8)
- added Cx3: 100nF, Capacitor_THT:C_Disc_D5.0mm_W2.5mm_P5.00mm, F.Cu at (-86.0, 130.8)
- added D1: 1N5819, Diode_THT:D_DO-41_SOD81_P10.16mm_Horizontal, F.Cu at (-36.7, 102.5)
- added D2: 1N5819, Diode_THT:D_DO-41_SOD81_P10.16mm_Horizontal, F.Cu at (-36.7, 106.8)
- added D3: 1N5819, Diode_THT:D_DO-41_SOD81_P10.16mm_Horizontal, F.Cu at (-36.7, 111.0)
- added D4: 1N5819, Diode_THT:D_DO-41_SOD81_P10.16mm_Horizontal, F.Cu at (-36.7, 115.3)
- added D5: 1N5819, Diode_THT:D_DO-41_SOD81_P10.16mm_Horizontal, F.Cu at (-36.7, 119.5)
- added D6: 1N5819, Diode_THT:D_DO-41_SOD81_P10.16mm_Horizontal, F.Cu at (-36.7, 123.8)
- added J3: Conn_01x02_Pin, TerminalBlock_Phoenix:TerminalBlock_Phoenix_MKDS-1,5-2_1x02_P5.00mm_Horizontal, F.Cu at (-62.5, 126.5)
- added L3: 680nH, xmitter:T68-6_Flat_HandWound, F.Cu at (-76.0, 77.2)
- added L5: 790nH, xmitter:T68-6_Vertical_HandWound, F.Cu at (-30.4, 71.2)
- added L8: 680nH, xmitter:T68-6_Flat_HandWound, F.Cu at (-53.0, 77.2)
- added Q2: 40673, Package_TO_SOT_THT:TO-72-4, F.Cu at (-76.5, 132.9)
- added Q3: 2N3904, Package_TO_SOT_THT:TO-92_Inline_Wide, F.Cu at (-25.5, 129.2)
- added Q8: 2N3904, Package_TO_SOT_THT:TO-92_Inline_Wide, F.Cu at (-25.5, 135.0)
- added R19: 10R, Resistor_THT:R_Axial_DIN0207_L6.3mm_D2.5mm_P10.16mm_Horizontal, F.Cu at (-77.8, 102.5)
- added R20: 1K5, Resistor_THT:R_Axial_DIN0207_L6.3mm_D2.5mm_P10.16mm_Horizontal, F.Cu at (-77.8, 106.5)
- added RP4: 62R, Resistor_THT:R_Axial_DIN0207_L6.3mm_D2.5mm_P10.16mm_Horizontal, F.Cu at (-77.8, 110.5)
- added RP5: 240R, Resistor_THT:R_Axial_DIN0207_L6.3mm_D2.5mm_P10.16mm_Horizontal, F.Cu at (-77.8, 114.6)
- added RP6: 62R, Resistor_THT:R_Axial_DIN0207_L6.3mm_D2.5mm_P10.16mm_Horizontal, F.Cu at (-77.8, 118.7)
- added RS2: 0R, Resistor_THT:R_Axial_DIN0207_L6.3mm_D2.5mm_P10.16mm_Horizontal, F.Cu at (-77.8, 122.7)
- added RT2: 50R, Resistor_THT:R_Axial_DIN0207_L6.3mm_D2.5mm_P10.16mm_Horizontal, F.Cu at (-77.8, 126.8)
- added TP24: +5V, Connector_PinHeader_2.54mm:PinHeader_1x01_P2.54mm_Vertical, F.Cu at (-42.1, 96.8)
- added U10: LM7171xIN, Package_DIP:DIP-8_W7.62mm, F.Cu at (-75.2, 90.8)
- added U11: LM7171xIN, Package_DIP:DIP-8_W7.62mm, F.Cu at (-64.4, 90.8)
- added U12: LM7171xIN, Package_DIP:DIP-8_W7.62mm, F.Cu at (-53.6, 90.8)
- added U13: LM7812_TO220, Package_TO_SOT_THT:TO-220-3_Vertical, F.Cu at (-35.4, 129.8)
- added U14: LM317L_TO92, Package_TO_SOT_THT:TO-92_Inline, F.Cu at (-42.4, 92.0)
- added U22: LM7805_TO220, Package_TO_SOT_THT:TO-220-3_Vertical, F.Cu at (-35.4, 135.8)
- added U5: Si5351A_Breakout, xmitter:Adafruit_Si5351A_STEMMA, F.Cu at (-52.3, 110.3)
- added U9: MCP4921, Package_DIP:DIP-8_W7.62mm, F.Cu at (-85.9, 90.8)
- J5: value ENC_INT if needed -> Conn_01x02_Pin; footprint xmitter:SameSky_RCJ-02_RCA_Jack -> TerminalBlock_Phoenix:TerminalBlock_Phoenix_MKDS-1,5-2_1x02_P5.00mm_Horizontal
- Q4, Q5, Q6, Q7: footprint Package_TO_SOT_THT:TO-92_Inline -> Package_TO_SOT_THT:TO-92_Inline_Wide
- moved J5 207.3 mm to (-50.5, 126.5), turned to 0 degrees
Connections:
- J4 pad 5: GND -> ENC_INT
- J5 pad 1: Net-(J5-In) -> +12V
- J5 pad 2: GND -> -12V
- R102 pad 2: Net-(J5-In) -> ENC_INT
- U16 pad 1: Net-(U16-1Y) -> MBL_A_N
- U16 pad 3: MBL_A_N -> Net-(U16-1Y)
- U17 pad P7: unconnected-(U17-PadP7) -> KeyUp
- U18 pad 11: +5V -> GND
- U18 pad 13: GND -> +5V
- U18 pad 3: GND -> +5V
- U18 pad 5: +5V -> GND
Routing:
- net (no net): track 0.00 -> 1642.0 mm, vias 0 -> 8
- net VEE: track 197.0 -> 0.00 mm, vias 3 -> 0
- net VA_INJ: track 144.7 -> 0.00 mm
- net VB_INJ: track 135.3 -> 0.00 mm
- net T1_COL: track 89.8 -> 0.00 mm
- net Net-(U3-CAR_IN-): track 86.3 -> 0.00 mm
- net Net-(U3-SIG_IN+): track 82.0 -> 0.00 mm, vias 2 -> 0
- net Net-(U6-+): track 70.6 -> 0.00 mm, vias 1 -> 0
- net Net-(CF5-Pad1): track 65.2 -> 0.00 mm
- net MC_OUT-: track 63.1 -> 0.00 mm
- net T2_COL: track 57.0 -> 0.00 mm
- net Net-(U7-+): track 42.9 -> 0.00 mm
- net RAW_RF: track 40.6 -> 0.00 mm, vias 1 -> 0
- net Net-(U3-SIG_IN-): track 39.0 -> 0.00 mm
- net Net-(CF3-Pad1): track 38.0 -> 0.00 mm
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
Commit message: KiCad revB: reset analog PCB to blank slate for fresh layout
Stripped all layout content from analog.kicad_pcb:
- 80 footprints
- 698 orphaned track segments (F.Cu, unnamed nets from before the
  VFO/VFO_Buffer_keyer sheet removal)
- 18 vias, 2 GND zones (F.Cu + B.Cu pours)
- 1 gr_rect, 1 gr_text

Preserved: version, generator, general (1.6 mm thickness), paper,
24-layer definition set, full setup block (FR4 stackup with 1.51 mm
core / 0.035 mm copper, tenting, plot parameters targeting gerber/).
Default (net 0 "") re-inserted.

File shrinks from ~43 kLOC to 131 lines. Ready for Update PCB from
Schematic to re-import footprints as an unrouted cloud.

Co-Authored-By: Claude Opus 4.7 <noreply@anthropic.com>
Parts:
- removed C24, C34, C36, C38, C42, Cx2, Cx3: 100nF, Capacitor_THT:C_Disc_D5.0mm_W2.5mm_P5.00mm
- removed C25, C35, C37, C43, C87: 10uF, Capacitor_THT:CP_Radial_D5.0mm_P2.00mm
- removed C27: 10uF, Capacitor_THT:C_Rect_L7.2mm_W4.5mm_P5.00mm
- removed C28, C41: 1uF, Capacitor_THT:C_Rect_L7.2mm_W4.5mm_P5.00mm
- removed C29: 680nF, Capacitor_THT:C_Rect_L13.0mm_W6.0mm_P10.00mm_FKS3_FKP3_MKS4
- removed C85: 0.33uF, Capacitor_THT:C_Rect_L7.0mm_W3.5mm_P5.00mm
- removed C86: 0.1uF, Capacitor_THT:C_Disc_D5.0mm_W2.5mm_P5.00mm
- removed CC2, C_IN4: 10nF, Capacitor_THT:C_Disc_D5.0mm_W2.5mm_P5.00mm
- removed CF2, CF8: 220pF, Capacitor_THT:C_Disc_D6.0mm_W2.5mm_P5.00mm
- removed CF4, CF6: 390pF, Capacitor_THT:C_Disc_D7.5mm_W2.5mm_P5.00mm
- removed D1, D2, D3, D4, D5, D6: 1N5819, Diode_THT:D_DO-41_SOD81_P10.16mm_Horizontal
- removed J15: Conn_01x03_Pin, Connector_PinHeader_2.54mm:PinHeader_1x03_P2.54mm_Vertical
- removed J3, J5: Conn_01x02_Pin, TerminalBlock_Phoenix:TerminalBlock_Phoenix_MKDS-1,5-2_1x02_P5.00mm_Horizontal
- removed J4: 8P8C_Shielded, xmitter:Amphenol_RJE1D-188_Horizontal_Shielded
- removed J6: TX/RX, Connector_PinHeader_2.54mm:PinHeader_1x02_P2.54mm_Vertical
- removed J7: HV, Connector_PinHeader_2.54mm:PinHeader_1x02_P2.54mm_Vertical
- removed J8: HV_INRUSH_BYPASS, Connector_PinHeader_2.54mm:PinHeader_1x02_P2.54mm_Vertical
- removed J9: TR_SENSE, Connector_PinHeader_2.54mm:PinHeader_1x02_P2.54mm_Vertical
- removed L3, L8: 680nH, xmitter:T68-6_Flat_HandWound
- removed L5: 790nH, xmitter:T68-6_Vertical_HandWound
- removed Q2: 40673, Package_TO_SOT_THT:TO-72-4
- removed Q3, Q8: 2N3904, Package_TO_SOT_THT:TO-92_Inline_Wide
- removed Q4, Q5, Q6, Q7: 2N7000, Package_TO_SOT_THT:TO-92_Inline_Wide
- removed R100, R101: 120, Resistor_THT:R_Axial_DIN0207_L6.3mm_D2.5mm_P10.16mm_Horizontal
- removed R102, R28, R29: 10K, Resistor_THT:R_Axial_DIN0207_L6.3mm_D2.5mm_P10.16mm_Horizontal
- removed R19: 10R, Resistor_THT:R_Axial_DIN0207_L6.3mm_D2.5mm_P10.16mm_Horizontal
- removed R20: 1K5, Resistor_THT:R_Axial_DIN0207_L6.3mm_D2.5mm_P10.16mm_Horizontal
- removed R26, R27: 2.2K, Resistor_THT:R_Axial_DIN0207_L6.3mm_D2.5mm_P10.16mm_Horizontal
- removed R30: 470K, Resistor_THT:R_Axial_DIN0207_L6.3mm_D2.5mm_P10.16mm_Horizontal
- removed RP4, RP6: 62R, Resistor_THT:R_Axial_DIN0207_L6.3mm_D2.5mm_P10.16mm_Horizontal
- removed RP5: 240R, Resistor_THT:R_Axial_DIN0207_L6.3mm_D2.5mm_P10.16mm_Horizontal
- removed RS2: 0R, Resistor_THT:R_Axial_DIN0207_L6.3mm_D2.5mm_P10.16mm_Horizontal
- removed RT2: 50R, Resistor_THT:R_Axial_DIN0207_L6.3mm_D2.5mm_P10.16mm_Horizontal
- removed TP11: Heartbeat, Connector_PinHeader_2.54mm:PinHeader_1x01_P2.54mm_Vertical
- removed TP16: TX/RX, Connector_PinHeader_2.54mm:PinHeader_1x01_P2.54mm_Vertical
- removed TP17: HV, Connector_PinHeader_2.54mm:PinHeader_1x01_P2.54mm_Vertical
- removed TP18: Inrush, Connector_PinHeader_2.54mm:PinHeader_1x01_P2.54mm_Vertical
- removed TP19: HB trigger, Connector_PinHeader_2.54mm:PinHeader_1x01_P2.54mm_Vertical
- removed TP24: +5V, Connector_PinHeader_2.54mm:PinHeader_1x01_P2.54mm_Vertical
- removed U10, U11, U12: LM7171xIN, Package_DIP:DIP-8_W7.62mm
- removed U13: LM7812_TO220, Package_TO_SOT_THT:TO-220-3_Vertical
- removed U14: LM317L_TO92, Package_TO_SOT_THT:TO-92_Inline
- removed U16: AM26LS32ACN, Package_DIP:DIP-16_W7.62mm
- removed U17: Adafruit_PCF8575_Breakout, xmitter:Adafruit_PCF8575_Breakout
- removed U18: CD14538B, Package_DIP:DIP-16_W7.62mm
- removed U22: LM7805_TO220, Package_TO_SOT_THT:TO-220-3_Vertical
- removed U5: Si5351A_Breakout, xmitter:Adafruit_Si5351A_STEMMA
- removed U9: MCP4921, Package_DIP:DIP-8_W7.62mm
Routing:
- net (no net): track 1642.0 -> 0.00 mm, vias 8 -> 0
- net +12V: track 341.1 -> 0.00 mm, vias 2 -> 0
- net +5V: track 305.8 -> 0.00 mm, vias 3 -> 0
- net 3V3: track 259.1 -> 0.00 mm, vias 1 -> 0
- net SDA: track 231.9 -> 0.00 mm
- net SCL: track 165.4 -> 0.00 mm, vias 1 -> 0
- net Net-(U18-+TR_A): track 72.7 -> 0.00 mm
- net MBL_A_P: track 58.6 -> 0.00 mm
- net MBL_A_N: track 53.8 -> 0.00 mm, vias 2 -> 0
- net Net-(Q6-G): track 53.2 -> 0.00 mm
- net Net-(Q5-G): track 44.5 -> 0.00 mm
- net Net-(Q4-G): track 40.6 -> 0.00 mm
- net MBL600_A: track 34.8 -> 0.00 mm
- net MBL_B_P: track 34.2 -> 0.00 mm
- net MBL_B_N: track 33.7 -> 0.00 mm, vias 1 -> 0
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- removed copper zone on B.Cu, net GND
- removed copper zone on F.Cu, net GND
Other:
- board outline removed
- board text removed: "Rev A"

Commit message: KiCad revC: analog PCB 9x7 landscape outline + 4x M3 mounting holes
Set up the empty analog PCB with:
- 9" x 7" landscape Edge.Cuts rectangle (228.60 x 177.80 mm) at (20, 20)
- 2 mm Margin inset as component keep-out visual indicator
- Four M3 NPTH mounting holes (H1..H4) 5 mm inboard from each corner,
  matching the frontpanel.kicad_pcb mounting-hole footprint style
- Paper switched to A3 so the drawing sheet comfortably surrounds the board

analog.net refresh is cosmetic: KiCad regenerated the Footprint-field
s-expr form; no footprint assignments changed.

Co-Authored-By: Claude Opus 4.7 <noreply@anthropic.com>
Parts:
- added H1: MountingHole_3.2mm_M3, MountingHole:MountingHole_3.2mm_M3, F.Cu at (25.0, 25.0)
- added H2: MountingHole_3.2mm_M3, MountingHole:MountingHole_3.2mm_M3, F.Cu at (243.6, 25.0)
- added H3: MountingHole_3.2mm_M3, MountingHole:MountingHole_3.2mm_M3, F.Cu at (25.0, 192.8)
- added H4: MountingHole_3.2mm_M3, MountingHole:MountingHole_3.2mm_M3, F.Cu at (243.6, 192.8)
Other:
- board outline added: 228.6 x 177.8 mm

Commit message: revD: analog board — DGFET+RC+buffer chain, LPF moved to ss_pa, PCB resized
Architecture change motivated by the Rev C sim finding that the LM7171
PP driver's +/-12V rails capped clean output at ~4.5W (see commit
3ce203d). Rev D delegates the gain-driver job to an external PA stage
(expected: QRP Labs 10W kit), so the analog board now just:
  Si5351 -> DGFET keyer -> R1(50)+C1(100p) RC @ 32MHz
         -> U1 LM7171 unity-gain follower -> R2(50) back-match -> J1 coax

Analog board changes (vfo_complete.kicad_sch):
  * DELETED: U10, U11, U12 (LM7171 PP driver chain) + feedback R/C,
    AC-coupling caps, V_BIAS network, R_GA/R_GB, C_GA/C_GB, J3/J4
    (dual-ended PP coax outputs)
  * DELETED: U2 reconstruction LPF stage (part of lpf.kicad_sch which
    is now emptied -- content moved to ss_pa/lpf.kicad_sch)
  * ADDED: R1=50R + C1=100pF (32 MHz single-pole RC snubber at the
    DGFET drain), U1 LM7171 unity-gain follower, R2=50R output
    back-match, J1 Conn_Coaxial_Small (new single-ended RF output),
    C2/C3=100nF op-amp bypass caps

Arduino sheet (arduino.kicad_sch):
  * ADDED: J2 Amphenol RJE1D-188 RJ45 for new external LPF board
    - Pins 1,2,3,6: RLY_10/15/17/20 band-select signals from PCF8575
    - Pins 5,8: GRID_CTL_A/B reserved spares for potential future
      tube PA (no other destination on the board, intentional)
    - Pins 4,7,SH: GND
  * ADDED: RLY_40 provision (not yet routed to J2, provision only)
  * T568B wire-pair arrangement for noise immunity

LPF content moved from analog/lpf.kicad_sch -> ss_pa/lpf.kicad_sch
(empty analog LPF sheet remains as a shell; delete later or repurpose).

PCB (analog.kicad_pcb):
  * Resized board outline from oversized 228x178 mm to 200x150 mm
    landscape (300 cm^2 / 46.5 in^2), centered on A3 at (210, 148.5)
  * Four M3 mounting holes H1-H4 placed 5 mm in from each corner
    (hole span 190 x 140 mm)
  * Added "board_only" attribute to each mounting hole so KiCad no
    longer flags them for deletion in Update PCB f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
Parts:
- moved H1 104.7 mm to (115.0, 78.5)
- moved H3 93.6 mm to (115.0, 218.5)
- moved H2 81.4 mm to (305.0, 78.5)
- moved H4 66.6 mm to (305.0, 218.5)
Other:
- board size 228.6 x 177.8 mm -> 200 x 150 mm
Changed lines of the file:
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@@
 	(net 0 "")
 	(gr_rect
-		(start 20 20)
-		(end 248.60 197.80)
+		(start 110 73.5)
+		(end 310 223.5)
 		(stroke
 			(width 0.15)
@@
 	)
 	(gr_rect
-		(start 22 22)
-		(end 246.60 195.80)
+		(start 112 75.5)
+		(end 308 221.5)
 		(stroke
 			(width 0.1)
@@
 	(footprint "MountingHole:MountingHole_3.2mm_M3"
 		(layer "F.Cu")
-		(at 25 25)
+		(at 115 78.5)
 		(descr "Mounting Hole 3.2mm, M3, no annular")
 		(tags "mountinghole M3")
@@
 			)
 		)
-		(attr exclude_from_pos_files exclude_from_bom)
+		(attr board_only exclude_from_pos_files exclude_from_bom)
 		(duplicate_pad_numbers_are_jumpers no)
 		(fp_circle
@@
 	(footprint "MountingHole:MountingHole_3.2mm_M3"
 		(layer "F.Cu")
-		(at 243.60 25)
+		(at 305 78.5)
 		(descr "Mounting Hole 3.2mm, M3, no annular")
 		(tags "mountinghole M3")
@@
 			)
 		)
-		(attr exclude_from_pos_files exclude_from_bom)
+		(attr board_only exclude_from_pos_files exclude_from_bom)
 		(duplicate_pad_numbers_are_jumpers no)
 		(fp_circle
@@
 	(footprint "MountingHole:MountingHole_3.2mm_M3"
 		(layer "F.Cu")
-		(at 25 192.80)
+		(at 115 218.5)
 		(descr "Mounting Hole 3.2mm, M3, no annular")
 		(tags "mountinghole M3")
@@
 			)
 		)
-		(attr exclude_from_pos_files exclude_from_bom)
+		(attr board_only exclude_from_pos_files exclude_from_bom)
 		(duplicate_pad_numbers_are_jumpers no)
 		(fp_circle
@@
 	(footprint "MountingHole:MountingHole_3.2mm_M3"
 		(layer "F.Cu")
-		(at 243.60 192.80)
+		(at 305 218.5)
 		(descr "Mounting Hole 3.2mm, M3, no annular")
 		(tags "mountinghole M3")
@@
 			)
 		)
-		(attr exclude_from_pos_files exclude_from_bom)
+		(attr board_only exclude_from_pos_files exclude_from_bom)
 		(duplicate_pad_numbers_are_jumpers no)
 		(fp_circle
