File: KiCAD/analog/dac.kicad_sch (KiCad schematic)
At the start: 17 parts, among them Q11 2N3904, Q12 2N3904, U4 MCP4922-EP

Commit message: revD analog: I2C level shifter for M6 + xmitter library additions
- Add Adafruit #757 BSS138 4-channel bidirectional I2C level shifter
  at the Si5351 I2C entry point on analog. Metro drives LV1/LV2 at
  +3.3V, the shared I2C bus (U17 PCF8575 analog, PCF8575 + MCP4725
  frontpanel, Si5351, MCP4728) runs at +5V on the HV side.
- Local 0.1 uF decoupling at LV and HV pins of the breakout.
- xmitter library additions:
    * symbol:    Adafruit_757_LevelShifter (12-pin breakout, LV side
                 pins 1-6, HV side pins 7-12, pre-linked to footprint)
    * footprint: Adafruit_757_BSS138_LevelShifter (2x6 header pattern,
                 2.54 mm pitch, 12.7 mm row-to-row, 1.0 mm NPTH holes.
                 Row spacing VERIFY against physical stock before fab.)
- M7 fix: MCP4922 (U4) VDD moved to +3.3V so Metro's 3.3V SPI meets
  the DAC's logic-high threshold (V_IH = 0.7*VDD = 2.31V @ 3.3V, well
  below Metro's 3.3V output). V_REF <= 3.3V still ample for G2
  envelope and BS170 bias.

Co-Authored-By: Claude Opus 4.7 <noreply@anthropic.com>
Connections:
- net +5V: no longer C49.2, C50.1, R47.1, U4.1 (VDD)
- new net +3.3V: C49.2, C50.1, R47.1, U4.1 (VDD)
Changed lines of the file:
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@@
-	)
-	(symbol
-		(lib_id "power:+5V")
-		(at 120.65 50.8 270)
-		(unit 1)
-		(body_style 1)
-		(exclude_from_sim no)
-		(in_bom yes)
-		(on_board yes)
-		(in_pos_files yes)
-		(dnp no)
-		(fields_autoplaced yes)
-		(property "Reference" "#PWR0116"
-			(at 116.84 50.8 0)
-			(hide yes)
-			(show_name no)
-			(do_not_autoplace no)
-			(effects
-				(font
-					(size 1.27 1.27)
-				)
-			)
-		)
-		(property "Value" "+5V"
-			(at 124.46 50.7999 90)
-			(show_name no)
-			(do_not_autoplace no)
-			(effects
-				(font
-					(size 1.27 1.27)
-				)
-				(justify left)
-			)
-		)
-		(property "Footprint" ""
-			(at 120.65 50.8 0)
-			(hide yes)
-			(show_name no)
-			(do_not_autoplace no)
-			(effects
-				(font
-					(size 1.27 1.27)
-				)
-			)
-		)
-		(property "Datasheet" ""
-			(at 120.65 50.8 0)
-			(hide yes)
-			(show_name no)
-			(do_not_autoplace no)
-			(effects
-				(font
-					(size 1.27 1.27)
-				)
-			)
-		)
-		(property "Description" "Power symbol creates a global label with name \"+5V\""
-			(at 120.65 50.8 0)
-			(hide yes)
-			(show_name no)
-			(do_not_autoplace no)
-			(effects
-				(font
-					(size 1.27 1.27)
-				)
-			)
-		)
-		(pin "1"
-		)
-		(instances
-			(project "analog"
-				(path "/d3de40b8-856b-4fbd-829c-f45ffcd55742/e880f7dd-82a1-4efe-84f5-e6a9d5641736"
-					(reference "#PWR0116")
-					(unit 1)
-				)
-			)
-		)
 	)
 	(symbol
@@
 					(unit 1)
 				)
+			)
+		)
+	)
+	(symbol
+		(lib_id "power:+3.3V")
+		(at 120.65 50.8 270)
+		(unit 1)
+		(body_style 1)
+		(exclude_from_sim no)
+		(in_bom yes)
+		(on_board yes)
+		(in_pos_files yes)
+		(dnp no)
+		(fields_autoplaced yes)
+		(property "Reference" "#PWR038"
+			(at 116.84 50.8 0)
+			(hide yes)
+			(show_name no)
+			(do_not_autoplace no)
+			(effects
+				(font
+					(size 1.27 1.27)
+				)
+			)
+		)
+		(property "Value" "+3.3V"
+			(at 124.46 50.7999 90)
+			(show_name no)
+			(do_not_autoplace no)
+			(effects
+				(font
+					(size 1.27 1.27)
+				)
+				(justify left)
+			)
+		)
+		(property "Footprint" ""
+			(at 120.65 50.8 0)
+			(hide yes)
+			(show_name no)
+			(do_not_autoplace no)
+			(effects
+				(font
+					(size 1.27 1.27)
+				)
+			)
+		)
+		(property "Datasheet" ""
+			(at 120.65 50.8 0)
+			(hide yes)
+			(show_name no)
+			(do_not_autoplace no)
+			(effects
+				(font
+					(size 1.27 1.27)
+				)
+			)
+		)
+		(property "Description" "Power symbol creates a global label with name \"+3.3V\""
+			(at 120.65 50.8 0)
+			(hide yes)
+			(show_name no)
+			(do_not_autoplace no)
+			(effects
+				(font
+					(size 1.27 1.27)
+				)
+			)
+		)
+		(pin "1"
+		)
+		(instances
+			(project "analog"
+				(path "/d3de40b8-856b-4fbd-829c-f45ffcd55742/e880f7dd-82a1-4efe-84f5-e6a9d5641736"
+					(reference "#PWR038")
+					(unit 1)
+				)

Commit message: revD: ss_pa Option C 5V rail + analog SW1 THT + R/C footprints + doc refresh
ss_pa Option C: swap U13 to LM2936Z-5.0 (full +5V logic rail), re-size
R10 10K->6.8K to preserve ~0.3V fault trip at new rail, drop +3.3V net
entirely. Fixes the previously-dead +5V bus that had no source.

Analog SW1 (Si5351 bringup DPDT): swap SMD footprint for
Button_Switch_THT:SW_CK_JS202011CQN_DPDT_Straight. Verified pin-numbering
convention (pin 1 above pin 6 in THT) matches user's intended DPST
wiring; both SDA/SCL break together.

Analog: assign missing footprints to R3/R4/R5/R8/R9 (DIN0207 axial) and
C4/C5/C6/C7/C8 (disc ceramic 5mm). Add xmitter:DIP-14_W7.62mm.kicad_mod
and 74HCT125 symbol to the xmitter library.

Documentation: Rev D handoff doc updated with M1-M8 fix status, Option C
notes, I2C bus voltage architecture, 74HCT125 SPI shifter, FAULT_N
divider details, and Metro-no-footprint note. Supporting docs updated:
i2c_bus.md full rewrite for 5V HV bus + STEMMA reroute, revD_interconnect
board inventory refresh, status banners on ss_pa.md / Master_Description /
cw_envelope_keyer / front_panel_interface pointing to handoff doc for
items beyond their last-current date.

Co-Authored-By: Claude Opus 4.7 <noreply@anthropic.com>
Parts:
- added U9: 74HCT125, xmitter:DIP-14_W7.62mm, symbol xmitter:74HCT125
Connections:
- net +3.3V is gone; now on net +5V: C49.2, C50.1, R47.1, U4.1 (VDD)
- net +5V: now also U9.14 (VCC)
- net CS_DAC: now also U9.9; no longer U4.3 (~{CS})
- net DAC_LDAC_N: now also U9.12; no longer U4.8 (~{LDAC})
- net GND: now also U9.1, U9.10, U9.13, U9.4, U9.7 (GND)
- net MOSI: now also U9.2; no longer U4.5 (SDI)
- net SCK: now also U9.5; no longer U4.4 (SCK)
- new net: U4.3 (~{CS}), U9.8
- new net: U4.4 (SCK), U9.6
- new net: U4.5 (SDI), U9.3
- new net: U4.8 (~{LDAC}), U9.11
