File: KiCAD/analog/power.kicad_sch (KiCad schematic)
At the start: 35 parts, among them J33 Screw_Terminal_01x02, J34 Screw_Terminal_01x02, J5 Screw_Terminal_01x02, K5 G6RL-1-DC12, K6 G6RL-1-DC12, U13 MCP1700x-330xxTO, U6 LM2940CT-5.0, U7 LT1054, U8 LM2940CT-12

Commit message: revD: U18 heartbeat RC reset + fault_shutdown migrated to analog
- arduino.kicad_sch: R48 10K + C14 10uF RC on U18 RST_A holds
  CD14538B heartbeat watchdog in reset ~70-120ms during Metro boot,
  preventing SS_PWR_RLY / SS_PA_INRUSH false-energize while PCF8575
  defaults HIGH on its outputs
- fault_shutdown.kicad_sch (new): LM393 overcurrent trip +
  CD74HC4066 bias switch + V_REF latch migrated from ss_pa to
  analog so FAULT_N stays off the umbilical; co-located with the
  Metro that reads it. Ref numbers +200 to avoid collision with
  pre-existing analog refs
- analog.kicad_sch: adds Fault_Shutdown sub-sheet reference (page 11)
- ss_pa: fault_shutdown sheet reference removed; ss_pa.net reflects
  the component loss (eliminates ss_pa U3 LM2936 LDO and +5V rail
  dependency)
- pa_stage.kicad_sch: R1-R4 bumped to 2W (RSF200JT-73-0R22) with
  DIN0516 L15.5mm footprint; footprint cleanup pass
- power.kicad_sch: 4.7R dummy bumped to 4.7R 10W with Axial_Power
  L25.0mm W9.0mm P30.48mm footprint

Co-Authored-By: Claude Opus 4.7 <noreply@anthropic.com>
Parts:
- R42: value 4.7R -> 4.7R 10W; footprint Resistor_THT:R_Axial_DIN0207_L6.3mm_D2.5mm_P10.16mm_Horizontal -> Resistor_THT:R_Axial_Power_L25.0mm_W9.0mm_P30.48mm
Changed lines of the file:
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@@
 			)
 		)
-		(property "Value" "4.7R"
+		(property "Value" "4.7R 10W"
 			(at 46.99 158.75 90)
 			(show_name no)
@@
 			)
 		)
-		(property "Footprint" "Resistor_THT:R_Axial_DIN0207_L6.3mm_D2.5mm_P10.16mm_Horizontal"
+		(property "Footprint" "Resistor_THT:R_Axial_Power_L25.0mm_W9.0mm_P30.48mm"
 			(at 47.244 161.544 90)
 			(hide yes)
