File: KiCAD/ss_pa/lpf.kicad_sch (KiCad schematic)
At the start: 83 parts, among them J16 Screw_Terminal_01x02, J25 Screw_Terminal_01x02, J26 Screw_Terminal_01x02, J27 Screw_Terminal_01x02, J28 Filter In, K1 Relay_RSS-SR042P, K2 Relay_RSS-SR042P, K3 Relay_RSS-SR042P, K4 Relay_RSS-SR042P, Q1 2N7000, Q5 2N7000, Q8 2N7000, Q9 2N7000, U3 LM7171xIN

Commit message: revD: DGFET-DAC bias scheme, kit-style xfmr naming, custom footprints, Output LPF project
Architecture refinements since the previous revD commit (f8d7058):

Analog board (vfo_complete, arduino, dac, power sheets):
  * MCP4922 (U4) ch B exposed as DRIVER_BIAS DAC output -> J31 pin 6
    (replaces the +3.3V pin that was on J31 pin 6 before). Analog's U4
    now controls the ss_pa BS170 driver DC bias point directly from
    firmware -- cleaner than the kit's trimmer+Q201 scheme.
  * MCP4728 (U3) ch A/B exposed as PA_Bias_A_Raw / PA_Bias_B_Raw ->
    J31 pins 7, 8. These feed the ss_pa CD74HC4066 fault-switch (U2),
    which gates them to PA_Bias_A/B on the IRF510 gates. On FAULT_N
    low, switch opens -> IRF510 bias collapses -> conduction cuts.
  * Rename pass: Bias_A/B/_Raw labels -> PA_Bias_A/B/_Raw everywhere
    (analog J3 screw-terminal, umbilical J31, ss_pa U2 inputs). Prefix
    disambiguates from DRIVER_BIAS which drives a different stage.
  * J2 (band-select RJ45 to Output LPF board): added RLY_40 provision.
    Pin layout reorganized -- RLY_40 lives at pin 5, pin 6 kept as a
    spare for a future 6th band.

ss_pa board (pa_stage, fault_shutdown, lpf sheets):
  * Driver + final BS170/IRF510 topology drawn following QRP Labs
    10W Linear kit (RF IN -> T201 input xfmr -> BS170 PP driver
    (Q2, Q6) -> T202 interstage -> IRF510 PP finals (Q3, Q4) ->
    T203 bifilar drain feed -> T204 output xfmr -> RF out).
  * Transformer references renamed to match the kit: T201 (input,
    BN61-2402), T202 (interstage, BN61-2402), T203 (drain feed,
    T50-43), T204 (output, BN43-202).
  * Driver bias filter on DRIVER_BIAS: C19 (0.1uF) + C20 (100pF)
    bulk + HF bypass, into T201 secondary CT (pin 4).
  * +3.3V now locally regulated on ss_pa (MCP1700x-330xxTO, U13)
    from +13.8V, powering U1 (LM393) and U2 (CD74HC4066). J31
    pin 6 freed up for DRIVER_BIAS.
  * Duplicate RJ45 J7 deleted (was a leftover from pre-DAC-bias era).
  * J3 (SMA RF input from analog) foo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
Parts:
- removed C13: 10nF, Capacitor_THT:C_Disc_D6.0mm_W2.5mm_P5.00mm, symbol Device:C
- removed C16: 100nF, Capacitor_THT:C_Disc_D5.0mm_W2.5mm_P5.00mm, symbol Device:C
- removed C91, C96: 10uF, Capacitor_THT:CP_Radial_D5.0mm_P2.00mm, symbol Device:C_Polarized_US
- removed C93, C97: 100nF, Capacitor_THT:C_Disc_D5.0mm_W2.5mm_P5.00mm, symbol Device:C_US
- removed C94, C98: 10nF, Capacitor_THT:C_Disc_D6.0mm_W2.5mm_P5.00mm, symbol Device:C_US
- removed C95: 2pF, xmitter:C_Axial_Kemet_Aximax_C41X_L4.5mm_D2.6mm_P7.62mm_Horizontal, symbol Device:C_US
- removed CF10, CF13: 180pF, Capacitor_THT:C_Disc_D6.0mm_W2.5mm_P5.00mm, symbol Device:C
- removed CF11, CF12: 330pF, Capacitor_THT:C_Disc_D7.5mm_W2.5mm_P5.00mm, symbol Device:C
- removed CF14, CF17: 150pF, Capacitor_THT:C_Disc_D6.0mm_W2.5mm_P5.00mm, symbol Device:C
- removed CF15, CF16: 270pF, Capacitor_THT:C_Disc_D7.5mm_W2.5mm_P5.00mm, symbol Device:C
- removed CF18, CF21, CF23, CF24: 100pF, Capacitor_THT:C_Disc_D6.0mm_W2.5mm_P5.00mm, symbol Device:C
- removed CF19, CF20: 100pF, Capacitor_THT:C_Disc_D7.5mm_W2.5mm_P5.00mm, symbol Device:C
- removed CF22, CF25: 10pF, Capacitor_THT:C_Disc_D6.0mm_W2.5mm_P5.00mm, symbol Device:C
- removed CF3, CF9: 220pF, Capacitor_THT:C_Disc_D6.0mm_W2.5mm_P5.00mm, symbol Device:C
- removed CF5, CF7: 390pF, Capacitor_THT:C_Disc_D7.5mm_W2.5mm_P5.00mm, symbol Device:C
- removed D10, D7, D8, D9: 1N4148, Diode_THT:D_DO-35_SOD27_P7.62mm_Horizontal, symbol Diode:1N4148
- removed J16, J25, J26, J27: Screw_Terminal_01x02, TerminalBlock_Phoenix:TerminalBlock_Phoenix_MKDS-1,5-2_1x02_P5.00mm_Horizontal, symbol Connector:Screw_Terminal_01x02
- removed J28: Filter In, Connector_Coaxial:SMA_Amphenol_132134_Vertical, symbol Connector:Conn_Coaxial_Small
- removed K1, K2, K3, K4: Relay_RSS-SR042P, xmitter:Relay_SPST_RelComm_RSS-SR042P, symbol xmitter:Relay_SPST_RSS-SR042P
- removed L10: 599/576nH, 12T, xmitter:T50-6_Vertical_HandWound, symbol Device:L_Ferrite
- removed L11: 542/576nH 12T, xmitter:T50-6_Flat_HandWound, symbol Device:L_Ferrite
- removed L12, L14: 452/484nH, 11T, xmitter:T50-6_Flat_HandWound, symbol Device:L_Ferrite
- removed L13: 499/484nH, 11T, xmitter:T50-6_Vertical_HandWound, symbol Device:L_Ferrite
- removed L15, L17: 331/324nF, 9T, xmitter:T50-6_Flat_HandWound, symbol Device:L_Ferrite
- removed L16: 366/400nH, 10T, xmitter:T50-6_Vertical_HandWound, symbol Device:L_Ferrite
- removed L6, L9: 662/676nH, 13T, xmitter:T50-6_Vertical_HandWound, symbol Device:L_Ferrite
- removed L7: 542/576nH, 12T, xmitter:T50-6_Flat_HandWound, symbol Device:L_Ferrite
- removed L8: 733/784nH, 14T, xmitter:T50-6_Flat_HandWound, symbol Device:L_Ferrite
- removed Q1, Q5, Q8, Q9: 2N7000, Package_TO_SOT_THT:TO-92_Inline, symbol Transistor_FET:2N7000
- removed R12, R42: 1K, Resistor_THT:R_Axial_DIN0207_L6.3mm_D2.5mm_P10.16mm_Horizontal, symbol Device:R_US
- removed R43: 4.7K, Resistor_THT:R_Axial_DIN0207_L6.3mm_D2.5mm_P10.16mm_Horizontal, symbol Device:R_US
- removed RP10, RP12, RP13, RP15, RP16, RP18, RP7, RP9: 100R, Resistor_THT:R_Axial_DIN0207_L6.3mm_D2.5mm_P10.16mm_Horizontal, symbol Device:R_US
- removed RP11, RP14, RP17, RP8: 68R, Resistor_THT:R_Axial_DIN0207_L6.3mm_D2.5mm_P10.16mm_Horizontal, symbol Device:R_US
- removed RT3, RT4, RT5, RT6: 50R, Resistor_THT:R_Axial_DIN0207_L6.3mm_D2.5mm_P10.16mm_Horizontal, symbol Device:R_US
- removed TP10M1, TP15M1, TP17M1, TP20M1, TP7: TestPoint, Connector_PinHeader_2.54mm:PinHeader_1x01_P2.54mm_Vertical, symbol Connector:TestPoint
- removed U3: LM7171xIN, Package_DIP:DIP-8_W7.62mm, symbol Amplifier_Operational:LM7171xIN
Other:
- note removed: "All inductor values listed as Target/Actual, Turn ct Current value are for T50-6 toroid"

Commit message: revD: analog board — DGFET+RC+buffer chain, LPF moved to ss_pa, PCB resized
Architecture change motivated by the Rev C sim finding that the LM7171
PP driver's +/-12V rails capped clean output at ~4.5W (see commit
3ce203d). Rev D delegates the gain-driver job to an external PA stage
(expected: QRP Labs 10W kit), so the analog board now just:
  Si5351 -> DGFET keyer -> R1(50)+C1(100p) RC @ 32MHz
         -> U1 LM7171 unity-gain follower -> R2(50) back-match -> J1 coax

Analog board changes (vfo_complete.kicad_sch):
  * DELETED: U10, U11, U12 (LM7171 PP driver chain) + feedback R/C,
    AC-coupling caps, V_BIAS network, R_GA/R_GB, C_GA/C_GB, J3/J4
    (dual-ended PP coax outputs)
  * DELETED: U2 reconstruction LPF stage (part of lpf.kicad_sch which
    is now emptied -- content moved to ss_pa/lpf.kicad_sch)
  * ADDED: R1=50R + C1=100pF (32 MHz single-pole RC snubber at the
    DGFET drain), U1 LM7171 unity-gain follower, R2=50R output
    back-match, J1 Conn_Coaxial_Small (new single-ended RF output),
    C2/C3=100nF op-amp bypass caps

Arduino sheet (arduino.kicad_sch):
  * ADDED: J2 Amphenol RJE1D-188 RJ45 for new external LPF board
    - Pins 1,2,3,6: RLY_10/15/17/20 band-select signals from PCF8575
    - Pins 5,8: GRID_CTL_A/B reserved spares for potential future
      tube PA (no other destination on the board, intentional)
    - Pins 4,7,SH: GND
  * ADDED: RLY_40 provision (not yet routed to J2, provision only)
  * T568B wire-pair arrangement for noise immunity

LPF content moved from analog/lpf.kicad_sch -> ss_pa/lpf.kicad_sch
(empty analog LPF sheet remains as a shell; delete later or repurpose).

PCB (analog.kicad_pcb):
  * Resized board outline from oversized 228x178 mm to 200x150 mm
    landscape (300 cm^2 / 46.5 in^2), centered on A3 at (210, 148.5)
  * Four M3 mounting holes H1-H4 placed 5 mm in from each corner
    (hole span 190 x 140 mm)
  * Added "board_only" attribute to each mounting hole so KiCad no
    longer flags them for deletion in Update PCB f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
Parts:
- added C13: 10nF, Capacitor_THT:C_Disc_D6.0mm_W2.5mm_P5.00mm, symbol Device:C
- added C16: 100nF, Capacitor_THT:C_Disc_D5.0mm_W2.5mm_P5.00mm, symbol Device:C
- added C91, C96: 10uF, Capacitor_THT:CP_Radial_D5.0mm_P2.00mm, symbol Device:C_Polarized_US
- added C93, C97: 100nF, Capacitor_THT:C_Disc_D5.0mm_W2.5mm_P5.00mm, symbol Device:C_US
- added C94, C98: 10nF, Capacitor_THT:C_Disc_D6.0mm_W2.5mm_P5.00mm, symbol Device:C_US
- added C95: 2pF, xmitter:C_Axial_Kemet_Aximax_C41X_L4.5mm_D2.6mm_P7.62mm_Horizontal, symbol Device:C_US
- added CF10, CF13: 180pF, Capacitor_THT:C_Disc_D6.0mm_W2.5mm_P5.00mm, symbol Device:C
- added CF11, CF12: 330pF, Capacitor_THT:C_Disc_D7.5mm_W2.5mm_P5.00mm, symbol Device:C
- added CF14, CF17: 150pF, Capacitor_THT:C_Disc_D6.0mm_W2.5mm_P5.00mm, symbol Device:C
- added CF15, CF16: 270pF, Capacitor_THT:C_Disc_D7.5mm_W2.5mm_P5.00mm, symbol Device:C
- added CF18, CF21, CF23, CF24: 100pF, Capacitor_THT:C_Disc_D6.0mm_W2.5mm_P5.00mm, symbol Device:C
- added CF19, CF20: 100pF, Capacitor_THT:C_Disc_D7.5mm_W2.5mm_P5.00mm, symbol Device:C
- added CF22, CF25: 10pF, Capacitor_THT:C_Disc_D6.0mm_W2.5mm_P5.00mm, symbol Device:C
- added CF3, CF9: 220pF, Capacitor_THT:C_Disc_D6.0mm_W2.5mm_P5.00mm, symbol Device:C
- added CF5, CF7: 390pF, Capacitor_THT:C_Disc_D7.5mm_W2.5mm_P5.00mm, symbol Device:C
- added D10, D7, D8, D9: 1N4148, Diode_THT:D_DO-35_SOD27_P7.62mm_Horizontal, symbol Diode:1N4148
- added J16, J25, J26, J27: Screw_Terminal_01x02, TerminalBlock_Phoenix:TerminalBlock_Phoenix_MKDS-1,5-2_1x02_P5.00mm_Horizontal, symbol Connector:Screw_Terminal_01x02
- added J28: Filter In, Connector_Coaxial:SMA_Amphenol_132134_Vertical, symbol Connector:Conn_Coaxial_Small
- added K1, K2, K3, K4: Relay_RSS-SR042P, xmitter:Relay_SPST_RelComm_RSS-SR042P, symbol xmitter:Relay_SPST_RSS-SR042P
- added L10: 599/576nH, 12T, xmitter:T50-6_Vertical_HandWound, symbol Device:L_Ferrite
- added L11: 542/576nH 12T, xmitter:T50-6_Flat_HandWound, symbol Device:L_Ferrite
- added L12, L14: 452/484nH, 11T, xmitter:T50-6_Flat_HandWound, symbol Device:L_Ferrite
- added L13: 499/484nH, 11T, xmitter:T50-6_Vertical_HandWound, symbol Device:L_Ferrite
- added L15, L17: 331/324nF, 9T, xmitter:T50-6_Flat_HandWound, symbol Device:L_Ferrite
- added L16: 366/400nH, 10T, xmitter:T50-6_Vertical_HandWound, symbol Device:L_Ferrite
- added L6, L9: 662/676nH, 13T, xmitter:T50-6_Vertical_HandWound, symbol Device:L_Ferrite
- added L7: 542/576nH, 12T, xmitter:T50-6_Flat_HandWound, symbol Device:L_Ferrite
- added L8: 733/784nH, 14T, xmitter:T50-6_Flat_HandWound, symbol Device:L_Ferrite
- added Q1, Q5, Q8, Q9: 2N7000, Package_TO_SOT_THT:TO-92_Inline, symbol Transistor_FET:2N7000
- added R12, R42: 1K, Resistor_THT:R_Axial_DIN0207_L6.3mm_D2.5mm_P10.16mm_Horizontal, symbol Device:R_US
- added R43: 4.7K, Resistor_THT:R_Axial_DIN0207_L6.3mm_D2.5mm_P10.16mm_Horizontal, symbol Device:R_US
- added RP10, RP12, RP13, RP15, RP16, RP18, RP7, RP9: 100R, Resistor_THT:R_Axial_DIN0207_L6.3mm_D2.5mm_P10.16mm_Horizontal, symbol Device:R_US
- added RP11, RP14, RP17, RP8: 68R, Resistor_THT:R_Axial_DIN0207_L6.3mm_D2.5mm_P10.16mm_Horizontal, symbol Device:R_US
- added RT3, RT4, RT5, RT6: 50R, Resistor_THT:R_Axial_DIN0207_L6.3mm_D2.5mm_P10.16mm_Horizontal, symbol Device:R_US
- added TP10M1, TP15M1, TP17M1, TP20M1, TP7: TestPoint, Connector_PinHeader_2.54mm:PinHeader_1x01_P2.54mm_Vertical, symbol Connector:TestPoint
- added U3: LM7171xIN, Package_DIP:DIP-8_W7.62mm, symbol Amplifier_Operational:LM7171xIN
Connections:
- new net: C16.2, J28.1 (In), RP10.1, RP11.1, RP13.1, RP14.1, RP16.1, RP17.1, RP7.1, RP8.1
- new net: CF3.1, L6.1, RP8.2, RP9.1, TP20M1.1, TP7.1
- new net: CF19.1, CF23.1, L15.2, L16.1
- new net: CF7.1, L8.2, L9.1
- new net: CF9.1, K4.1 (RF_A), L9.2, RT3.1
- new net: D7.2 (A), J16.2 (Pin_2), Q1.3 (D)
- new net: CF5.1, L6.2, L8.1
- new net: C95.1, R42.1, R43.1, U3.2 (-)
- new net: C16.1, C95.2, R43.2, U3.6
- new net: CF14.1, L12.1, RP14.2, RP15.1, TP15M1.1
- new net: CF10.1, L7.1, RP11.2, RP12.1, TP17M1.1
- new net: CF18.1, CF22.1, L15.1, RP17.2, RP18.1, TP10M1.1
- new net: CF17.1, K2.1 (RF_A), L14.2, RT5.1
- new net: CF21.1, CF25.1, K1.1 (RF_A), L17.2, RT6.1
- new net: CF16.1, L13.2, L14.1
- new net: D10.2 (A), J27.2 (Pin_2), Q9.3 (D)
- new net: CF20.1, CF24.1, L16.2, L17.1
- new net: C13.2, R12.1, U3.3 (+)
- new net: CF11.1, L10.1, L7.2
- new net: CF15.1, L12.2, L13.1
- new net: D8.2 (A), J25.2 (Pin_2), Q5.3 (D)
- new net: CF13.1, K3.1 (RF_A), L11.2, RT4.1
- new net: CF12.1, L10.2, L11.1
- new net: D9.2 (A), J26.2 (Pin_2), Q8.3 (D)
- new net +12V: C96.1, C97.1, C98.1, U3.7 (V+)
- new net +28V: D10.1 (K), D7.1 (K), D8.1 (K), D9.1 (K), J16.1 (Pin_1), J25.1 (Pin_1), J26.1 (Pin_1), J27.1 (Pin_1)
- new net -12V: C91.1, C93.1, C94.1, U3.4 (V-)
- new net Conditioned RF: K1.2 (RF_B), K2.2 (RF_B), K3.2 (RF_B), K4.2 (RF_B)
- new net GND: C91.2, C93.2, C94.2, C96.2, C97.2, C98.2, CF10.2, CF11.2, CF12.2, CF13.2, CF14.2, CF15.2, CF16.2, CF17.2, CF18.2, CF19.2, CF20.2, CF21.2, CF22.2, CF23.2, CF24.2, CF25.2, CF3.2, CF5.2, CF7.2, CF9.2, J28.2 (Ext), K1.3 (SHIELD), K2.3 (SHIELD), K3.3 (SHIELD), K4.3 (SHIELD), Q1.1 (S), Q5.1 (S), Q8.1 (S), Q9.1 (S), R12.2, R42.2, RP10.2, RP12.2, RP13.2, RP15.2, RP16.2, RP18.2, RP7.2, RP9.2, RT3.2, RT4.2, RT5.2, RT6.2
- new net RLY_10: Q9.2 (G)
- new net RLY_15: Q5.2 (G)
- new net RLY_17: Q8.2 (G)
- new net RLY_20: Q1.2 (G)
- new net Raw RF: C13.1
Other:
- note added: "All inductor values listed as Target/Actual, Turn ct Current value are for T50-6 toroid"
